Commit message: refactor(ros): rename package four_bar_bot_description -> wojtek_description
Wojtek name convergence, ROS package #3 of 3 (ament_cmake). Atomic dir
move + full-token repoint; the 63 MB mesh set moves with the dir (git is
content-addressed, so blobs are reused, not re-stored).

  dir            ros/src/four_bar_bot_description/ -> ros/src/wojtek_description/
  package.xml    <name>four_bar_bot_description</name> -> wojtek_description
  CMakeLists.txt project(four_bar_bot_description)     -> wojtek_description

Consumers repointed (full token four_bar_bot_description only):
  - urdf xacros in this pkg (body/four_bar_bot/leg) $(find ...) + mesh paths
  - wojtek_bringup: package.xml depend, urdf/fbb_{real,sim}.xacro $(find),
    mujoco_sim_node get_package_share_directory()
  - ros/docker/Dockerfile colcon --packages-select
  - mujoco/check_model.py
  - training/fbb_rl/paths.py  MUJOCO_DIR (the cross-boundary ros<->training ref)

Deliberately NOT touched (separate tokens, later steps):
  - MJCF filenames four_bar_bot*.xml + four_bar_bot.urdf.xacro (step 3:
    MJCF rename). Model content byte-identical to baseline - verified in
    working tree against origin/main:quadruped_ros2_original/... (IDENTICAL).
  - *.md docs (plans/specs/package README) left as provenance.

verify.sh: repoint present-dir + paths.py grep + file-exists paths + the
equivalence RH (HEAD) side to wojtek_description; the QB baseline side
stays on origin/main's quadruped_ros2_original path so the check still
proves model byte-identity ACROSS the rename. T3 message updated, new T0
ghost guard "no live four_bar_bot_description ref".

Co-Authored-By: Claude Opus 4.8 (1M context) <noreply@anthropic.com>

File: ros/src/wojtek_bringup/urdf/fbb_real.urdf.xacro (robot description, xacro)
@@ -2,5 +2,5 @@
 <!--
   Real-robot URDF for running the RL policy.
-  Mechanically identical to four_bar_bot_description's four_bar_bot.urdf.xacro
+  Mechanically identical to wojtek_description's four_bar_bot.urdf.xacro
   (same leg macros), but the ros2_control block differs:
     * command interface `position` -> MD80 IMPEDANCE mode
@@ -12,5 +12,5 @@
 -->
 <robot name="quadruped" xmlns:xacro="http://www.ros.org/wiki/xacro">
-  <xacro:include filename="$(find four_bar_bot_description)/urdf/body.urdf.xacro" />
+  <xacro:include filename="$(find wojtek_description)/urdf/body.urdf.xacro" />
   <xacro:include filename="$(find wojtek_bringup)/urdf/fbb_ros2_control.urdf.xacro" />
   <xacro:arg name="kp" default="20.0" />

File: ros/src/wojtek_bringup/urdf/fbb_sim.urdf.xacro (robot description, xacro)
@@ -1,5 +1,5 @@
 <?xml version="1.0"?>
 <!--
-  Visualization/sim URDF: the same mechanics as four_bar_bot_description's
+  Visualization/sim URDF: the same mechanics as wojtek_description's
   four_bar_bot.urdf.xacro (base + imu + 4 legs) but without the ros2_control
   and Gazebo blocks. Physics comes from the MuJoCo sim node; this model
@@ -7,5 +7,5 @@
 -->
 <robot name="quadruped" xmlns:xacro="http://www.ros.org/wiki/xacro">
-  <xacro:include filename="$(find four_bar_bot_description)/urdf/body.urdf.xacro" />
+  <xacro:include filename="$(find wojtek_description)/urdf/body.urdf.xacro" />
   <xacro:four_bar_bot_body />
 </robot>

File: ros/src/wojtek_description/urdf/body.urdf.xacro (robot description, xacro)
@@ -1,6 +1,6 @@
 <?xml version="1.0"?>
 <robot xmlns:xacro="http://www.ros.org/wiki/xacro" name="four_bar_bot_body">
-  <xacro:include filename="$(find four_bar_bot_description)/urdf/inertia.urdf.xacro" />
-  <xacro:include filename="$(find four_bar_bot_description)/urdf/leg.urdf.xacro" />
+  <xacro:include filename="$(find wojtek_description)/urdf/inertia.urdf.xacro" />
+  <xacro:include filename="$(find wojtek_description)/urdf/leg.urdf.xacro" />
   <!-- Mechanical assembly shared by every bringup of this robot: material,
        base_link/body_link/imu_link, and the four legs. ros2_control/Gazebo
@@ -16,5 +16,5 @@
         <origin rpy="0 0 ${pi}" xyz="0.0 0 0" />
         <geometry name="base_link">
-          <mesh filename="package://four_bar_bot_description/meshes/base_link.dae" />
+          <mesh filename="package://wojtek_description/meshes/base_link.dae" />
         </geometry>
         <xacro:grey_material />
@@ -23,5 +23,5 @@
         <origin rpy="0 0 ${pi}" xyz="0.0 0 0" />
         <geometry name="base_link">
-          <mesh filename="package://four_bar_bot_description/meshes/base_link.dae" />
+          <mesh filename="package://wojtek_description/meshes/base_link.dae" />
         </geometry>
       </collision>

File: ros/src/wojtek_description/urdf/four_bar_bot.urdf.xacro (robot description, xacro)
@@ -1,9 +1,9 @@
 <?xml version="1.0"?>
 <robot name="quadruped" xmlns:xacro="http://www.ros.org/wiki/xacro">
-  <xacro:include filename="$(find four_bar_bot_description)/urdf/body.urdf.xacro" />
-  <xacro:include filename="$(find four_bar_bot_description)/urdf/ros2_control.urdf.xacro" />
-  <xacro:include filename="$(find four_bar_bot_description)/urdf/gazebo.urdf.xacro" />
+  <xacro:include filename="$(find wojtek_description)/urdf/body.urdf.xacro" />
+  <xacro:include filename="$(find wojtek_description)/urdf/ros2_control.urdf.xacro" />
+  <xacro:include filename="$(find wojtek_description)/urdf/gazebo.urdf.xacro" />
   <mujoco>
-    <compiler meshdir="$(find four_bar_bot_description)/meshes" balanceinertia="true"
+    <compiler meshdir="$(find wojtek_description)/meshes" balanceinertia="true"
       discardvisual="false" />
   </mujoco>

File: ros/src/wojtek_description/urdf/leg.urdf.xacro (robot description, xacro)
@@ -1,5 +1,5 @@
 <?xml version="1.0"?>
 <robot xmlns:xacro="http://www.ros.org/wiki/xacro" name="quadruped_robot">
-  <xacro:include filename="$(find four_bar_bot_description)/urdf/inertia.urdf.xacro" />
+  <xacro:include filename="$(find wojtek_description)/urdf/inertia.urdf.xacro" />
   <!-- Macro to define a leg -->
   <xacro:macro name="leg"
@@ -91,5 +91,5 @@
         <origin rpy="0 0 0" xyz="0.0 0 0.0" />
         <geometry>
-          <mesh filename="package://four_bar_bot_description/meshes/first_link.dae" />
+          <mesh filename="package://wojtek_description/meshes/first_link.dae" />
         </geometry>
         <xacro:grey_material />
@@ -98,5 +98,5 @@
         <origin rpy="0 0 0" xyz="0.0 0 0.0" />
         <geometry>
-          <mesh filename="package://four_bar_bot_description/meshes/first_link.dae" />
+          <mesh filename="package://wojtek_description/meshes/first_link.dae" />
         </geometry>
       </collision>
@@ -109,5 +109,5 @@
         <origin rpy="0 0 0" xyz="0.0 0 0.0" />
         <geometry>
-          <mesh filename="package://four_bar_bot_description/meshes/second_link.dae" />
+          <mesh filename="package://wojtek_description/meshes/second_link.dae" />
         </geometry>
         <xacro:grey_material />
@@ -116,5 +116,5 @@
         <origin rpy="0 0 0" xyz="0.0 0 0.0" />
         <geometry>
-          <mesh filename="package://four_bar_bot_description/meshes/second_link.dae" />
+          <mesh filename="package://wojtek_description/meshes/second_link.dae" />
         </geometry>
       </collision>
@@ -127,5 +127,5 @@
         <origin rpy="0 0 0" xyz="0.0 0 0.0" />
         <geometry>
-          <mesh filename="package://four_bar_bot_description/meshes/third_link.dae" />
+          <mesh filename="package://wojtek_description/meshes/third_link.dae" />
         </geometry>
         <xacro:grey_material />
@@ -134,5 +134,5 @@
         <origin rpy="0 0 0" xyz="0.0 0 0.0" />
         <geometry>
-          <mesh filename="package://four_bar_bot_description/meshes/third_link.dae" />
+          <mesh filename="package://wojtek_description/meshes/third_link.dae" />
         </geometry>
       </collision>
@@ -145,5 +145,5 @@
         <origin rpy="0 0 0" xyz="0.0 0 0.0" />
         <geometry>
-          <mesh filename="package://four_bar_bot_description/meshes/fourth_link.dae" />
+          <mesh filename="package://wojtek_description/meshes/fourth_link.dae" />
         </geometry>
         <xacro:grey_material />
@@ -152,5 +152,5 @@
         <origin rpy="0 0 0" xyz="0.0 0 0.0" />
         <geometry>
-          <mesh filename="package://four_bar_bot_description/meshes/fourth_link.dae" />
+          <mesh filename="package://wojtek_description/meshes/fourth_link.dae" />
         </geometry>
       </collision>
@@ -163,5 +163,5 @@
         <origin rpy="0 0 0" xyz="0.0 0 0.0" />
         <geometry>
-          <mesh filename="package://four_bar_bot_description/meshes/fifth_link.dae" />
+          <mesh filename="package://wojtek_description/meshes/fifth_link.dae" />
         </geometry>
         <xacro:grey_material />
@@ -170,5 +170,5 @@
         <origin rpy="0 0 0" xyz="0.0 0 0.0" />
         <geometry>
-          <mesh filename="package://four_bar_bot_description/meshes/fifth_link.dae" />
+          <mesh filename="package://wojtek_description/meshes/fifth_link.dae" />
         </geometry>
       </collision>
@@ -181,5 +181,5 @@
         <origin rpy="0 0 0" xyz="0.0 0 0.0" />
         <geometry>
-          <mesh filename="package://four_bar_bot_description/meshes/sixth_link.dae" />
+          <mesh filename="package://wojtek_description/meshes/sixth_link.dae" />
         </geometry>
         <xacro:grey_material />
@@ -188,5 +188,5 @@
         <origin rpy="0 0 0" xyz="0.0 0 0.0" />
         <geometry>
-          <mesh filename="package://four_bar_bot_description/meshes/sixth_link.dae" />
+          <mesh filename="package://wojtek_description/meshes/sixth_link.dae" />
         </geometry>
       </collision>
