Commit message: fix(md80): trzymaj pozę z aktywacji + prawdziwy no-torque w dry_run
Dwa fixy wokół bring-upu, oba potwierdzone na robocie:

1. Robot aktywnie odjeżdżał do "pozy supermana" przy starcie stacku.
   Komenda startowa ("trzymaj obecną pozycję") była zasiewana z odczytu
   zrobionego ZANIM initial_positions_ zostały zapamiętane, czyli w surowej
   ramce napędu; write() dodawał offset z powrotem i wysyłał 2x surową
   pozycję. Jeśli napędy miały niezerowe surowe zero (włączenie zasilania
   w innej pozie), robot w chwili enable jechał drugie tyle w tym samym
   kierunku. Fix: drugi read() po ustawieniu offsetów -- stan ~0, komenda
   staje się faktycznym "stój w miejscu".

2. --dry-run obiecywał "no torque", ale enable_motors() i tak uzbrajał
   napędy -- dry_run gate'ował tylko komendy w real_io_node, a jednorazowy
   target z on_activate szedł do silników z pełnym max_torque. Teraz launch
   przekazuje dry_run przez xacro do parametru <hardware> i przy dry_run
   drive'y nie są w ogóle enable'owane (controlMd80Enable pominięte,
   głośny WARN); candle->begin() dalej rusza, więc enkodery streamują
   i RViz/zero działają na benchu.

Do tego: imu_i2c_hardware_interface dodany jako depend wojtek_bringup
(deploy.sh --packages-up-to buduje go teraz na RPi) i do listy pakietów
budowanych w obrazie dev kontenera.

File: ros/src/wojtek_bringup/urdf/wojtek_real.urdf.xacro (robot description, xacro)
@@ -23,4 +23,7 @@
   <xacro:arg name="can_baud" default="8" />
   <xacro:arg name="usb_port" default="/dev/ttyACM0" />
+  <!-- Bench mode: drives are never enabled (no torque at all), encoder
+       states still stream. Set by the launches from their dry_run arg. -->
+  <xacro:arg name="dry_run" default="false" />
   <!-- The serial IMU (loaner BMI160 behind an MCU + CP2102 bridge) was retired
        2026-07-17 in favor of the Adafruit 5543 (LSM6DS3TR-C + LIS3MDL) wired
@@ -34,5 +37,6 @@
   <xacro:wojtek_body />
   <xacro:wojtek_ros2_control kp="$(arg kp)" kd="$(arg kd)" max_torque="$(arg max_torque)"
-    usb_port="$(arg usb_port)" bus="$(arg bus)" can_baud="$(arg can_baud)" />
+    usb_port="$(arg usb_port)" bus="$(arg bus)" can_baud="$(arg can_baud)"
+    dry_run="$(arg dry_run)" />
   <xacro:if value="$(arg use_imu)">
     <xacro:wojtek_imu_i2c_ros2_control bus="$(arg imu_bus)" addr_ag="$(arg imu_addr_ag)"

File: ros/src/wojtek_bringup/urdf/wojtek_ros2_control.urdf.xacro (robot description, xacro)
@@ -39,5 +39,5 @@
        8 since the 2026-07-17 migration for the HAT; the dongle setup ran 1.
        See ros/hw_tests/README.md for the per-drive baud migration tool. -->
-  <xacro:macro name="wojtek_ros2_control" params="kp kd max_torque usb_port bus:=spi can_baud:=8">
+  <xacro:macro name="wojtek_ros2_control" params="kp kd max_torque usb_port bus:=spi can_baud:=8 dry_run:=false">
     <ros2_control name="MD80HardwareInterface" type="system">
       <hardware>
@@ -46,4 +46,7 @@
         <param name="bus">${bus}</param>
         <param name="can_baud">${can_baud}</param>
+        <!-- true = bench mode: drives never enabled (no torque), encoder
+             states still stream. Wired from the launches' dry_run arg. -->
+        <param name="dry_run">${dry_run}</param>
       </hardware>
       <xacro:wojtek_joint name="front_left_first_joint" can_id="10" kp="${kp}" kd="${kd}" max_torque="${max_torque}" />
