Commit message: refactor(ros): rename urdf xacro files + macros fbb_*/four_bar_bot -> wojtek_*
Kill the fbb/four_bar_bot names in the URDF layer. Files:

  fbb_real.urdf.xacro         -> wojtek_real.urdf.xacro
  fbb_sim.urdf.xacro          -> wojtek_sim.urdf.xacro
  fbb_ros2_control.urdf.xacro -> wojtek_ros2_control.urdf.xacro
  four_bar_bot.urdf.xacro     -> wojtek.urdf.xacro   (wojtek_description)

Macros (def + every invocation, across both packages' xacros, the two
bringup launch files, real_controllers.yaml, and the bmi160 firmware README):

  four_bar_bot_body           -> wojtek_body
  fbb_joint                   -> wojtek_joint
  fbb_ros2_control            -> wojtek_ros2_control
  fbb_imu_ros2_control        -> wojtek_imu_ros2_control
  fbb_bmi160_imu_ros2_control -> wojtek_bmi160_imu_ros2_control

Also the real_io_node ROS node name "fbb_real_io" -> "wojtek_real_io"
(self-defined, no launch/param references it).

Deliberately untouched: the /fbb/* runtime service namespaces and the
fbb_loco_v8 policy name (open decisions on the PR), and the
<mujoco model="four_bar_bot"> attr (lives in mujoco/, a separate decision).

Verified: T0 45/0/0 with a new urdf-token ghost guard; T3 colcon build of
all 6 packages; and `xacro` expands both top-level bringup files in the
built image (wojtek_real 1128 lines, wojtek_sim 798 lines), so the full
macro tree and the cross-package description include resolve.

Co-Authored-By: Claude Opus 4.8 (1M context) <noreply@anthropic.com>

File: ros/src/wojtek_bringup/urdf/wojtek_real.urdf.xacro (robot description, xacro)
@@ -2,5 +2,5 @@
 <!--
   Real-robot URDF for running the RL policy.
-  Mechanically identical to wojtek_description's four_bar_bot.urdf.xacro
+  Mechanically identical to wojtek_description's wojtek.urdf.xacro
   (same leg macros), but the ros2_control block differs:
     * command interface `position` -> MD80 IMPEDANCE mode
@@ -13,5 +13,5 @@
 <robot name="quadruped" xmlns:xacro="http://www.ros.org/wiki/xacro">
   <xacro:include filename="$(find wojtek_description)/urdf/body.urdf.xacro" />
-  <xacro:include filename="$(find wojtek_bringup)/urdf/fbb_ros2_control.urdf.xacro" />
+  <xacro:include filename="$(find wojtek_bringup)/urdf/wojtek_ros2_control.urdf.xacro" />
   <xacro:arg name="kp" default="20.0" />
   <xacro:arg name="kd" default="1.0" />
@@ -20,5 +20,5 @@
   <!-- Loaner BMI160 (no magnetometer) until the real BMX160 is sourced;
        see bmi160_serial_hardware_interface. Swap back to
-       xacro:fbb_imu_ros2_control below once the real sensor is back.
+       xacro:wojtek_imu_ros2_control below once the real sensor is back.
        by-id path instead of /dev/ttyUSBx: the CP2102 drops off the bus on
        a flaky cable and can re-enumerate under a different number; the
@@ -27,11 +27,11 @@
   <xacro:arg name="imu_port"
     default="/dev/serial/by-id/usb-Silicon_Labs_CP2102_USB_to_UART_Bridge_Controller_0001-if00-port0" />
-  <xacro:four_bar_bot_body />
-  <xacro:fbb_ros2_control kp="$(arg kp)" kd="$(arg kd)" max_torque="$(arg max_torque)"
+  <xacro:wojtek_body />
+  <xacro:wojtek_ros2_control kp="$(arg kp)" kd="$(arg kd)" max_torque="$(arg max_torque)"
     usb_port="$(arg usb_port)" />
   <!-- IMU disabled: flaky BMI160 and fbb_loco_v8 doesn't observe it.
        Re-enable (with the imu_sensor_broadcaster in real_controllers.yaml
        and real.launch.py) before running an IMU-observing policy.
-  <xacro:fbb_bmi160_imu_ros2_control port="$(arg imu_port)" />
+  <xacro:wojtek_bmi160_imu_ros2_control port="$(arg imu_port)" />
   -->
 </robot>

File: ros/src/wojtek_bringup/urdf/wojtek_ros2_control.urdf.xacro (robot description, xacro)
@@ -6,5 +6,5 @@
        (wojtek_mjx.xml: gainprm=20, biasprm="0 -20 -1", forcerange 6)
        when kp=20, kd=1, max_torque=6. -->
-  <xacro:macro name="fbb_joint" params="name can_id kp kd max_torque">
+  <xacro:macro name="wojtek_joint" params="name can_id kp kd max_torque">
     <joint name="${name}">
       <command_interface name="position" />
@@ -34,5 +34,5 @@
     </joint>
   </xacro:macro>
-  <xacro:macro name="fbb_ros2_control" params="kp kd max_torque usb_port">
+  <xacro:macro name="wojtek_ros2_control" params="kp kd max_torque usb_port">
     <ros2_control name="MD80HardwareInterface" type="system">
       <hardware>
@@ -41,19 +41,19 @@
         <param name="bus">usb</param>
       </hardware>
-      <xacro:fbb_joint name="front_left_first_joint" can_id="10" kp="${kp}" kd="${kd}" max_torque="${max_torque}" />
-      <xacro:fbb_joint name="front_left_second_joint" can_id="11" kp="${kp}" kd="${kd}" max_torque="${max_torque}" />
-      <xacro:fbb_joint name="front_left_third_joint" can_id="12" kp="${kp}" kd="${kd}" max_torque="${max_torque}" />
-      <xacro:fbb_joint name="front_right_first_joint" can_id="20" kp="${kp}" kd="${kd}" max_torque="${max_torque}" />
-      <xacro:fbb_joint name="front_right_second_joint" can_id="21" kp="${kp}" kd="${kd}" max_torque="${max_torque}" />
-      <xacro:fbb_joint name="front_right_third_joint" can_id="22" kp="${kp}" kd="${kd}" max_torque="${max_torque}" />
-      <xacro:fbb_joint name="rear_right_first_joint" can_id="30" kp="${kp}" kd="${kd}" max_torque="${max_torque}" />
-      <xacro:fbb_joint name="rear_right_second_joint" can_id="31" kp="${kp}" kd="${kd}" max_torque="${max_torque}" />
-      <xacro:fbb_joint name="rear_right_third_joint" can_id="32" kp="${kp}" kd="${kd}" max_torque="${max_torque}" />
-      <xacro:fbb_joint name="rear_left_first_joint" can_id="40" kp="${kp}" kd="${kd}" max_torque="${max_torque}" />
-      <xacro:fbb_joint name="rear_left_second_joint" can_id="41" kp="${kp}" kd="${kd}" max_torque="${max_torque}" />
-      <xacro:fbb_joint name="rear_left_third_joint" can_id="42" kp="${kp}" kd="${kd}" max_torque="${max_torque}" />
+      <xacro:wojtek_joint name="front_left_first_joint" can_id="10" kp="${kp}" kd="${kd}" max_torque="${max_torque}" />
+      <xacro:wojtek_joint name="front_left_second_joint" can_id="11" kp="${kp}" kd="${kd}" max_torque="${max_torque}" />
+      <xacro:wojtek_joint name="front_left_third_joint" can_id="12" kp="${kp}" kd="${kd}" max_torque="${max_torque}" />
+      <xacro:wojtek_joint name="front_right_first_joint" can_id="20" kp="${kp}" kd="${kd}" max_torque="${max_torque}" />
+      <xacro:wojtek_joint name="front_right_second_joint" can_id="21" kp="${kp}" kd="${kd}" max_torque="${max_torque}" />
+      <xacro:wojtek_joint name="front_right_third_joint" can_id="22" kp="${kp}" kd="${kd}" max_torque="${max_torque}" />
+      <xacro:wojtek_joint name="rear_right_first_joint" can_id="30" kp="${kp}" kd="${kd}" max_torque="${max_torque}" />
+      <xacro:wojtek_joint name="rear_right_second_joint" can_id="31" kp="${kp}" kd="${kd}" max_torque="${max_torque}" />
+      <xacro:wojtek_joint name="rear_right_third_joint" can_id="32" kp="${kp}" kd="${kd}" max_torque="${max_torque}" />
+      <xacro:wojtek_joint name="rear_left_first_joint" can_id="40" kp="${kp}" kd="${kd}" max_torque="${max_torque}" />
+      <xacro:wojtek_joint name="rear_left_second_joint" can_id="41" kp="${kp}" kd="${kd}" max_torque="${max_torque}" />
+      <xacro:wojtek_joint name="rear_left_third_joint" can_id="42" kp="${kp}" kd="${kd}" max_torque="${max_torque}" />
     </ros2_control>
   </xacro:macro>
-  <xacro:macro name="fbb_imu_ros2_control" params="port baud_rate:=9600">
+  <xacro:macro name="wojtek_imu_ros2_control" params="port baud_rate:=9600">
     <ros2_control name="imu" type="sensor">
       <hardware>
@@ -79,10 +79,10 @@
     </ros2_control>
   </xacro:macro>
-  <!-- Loaner sensor stand-in for fbb_imu_ros2_control above: a bare BMI160
+  <!-- Loaner sensor stand-in for wojtek_imu_ros2_control above: a bare BMI160
        (accel+gyro only, no magnetometer) is what's actually wired in until
        a real BMX160 is sourced. See bmi160_serial_hardware_interface for
        why magnetometer.* is dropped: nothing downstream (imu_sensor_broadcaster,
        wojtek_policy) consumes it anyway. -->
-  <xacro:macro name="fbb_bmi160_imu_ros2_control" params="port baud_rate:=115200">
+  <xacro:macro name="wojtek_bmi160_imu_ros2_control" params="port baud_rate:=115200">
     <ros2_control name="imu" type="sensor">
       <hardware>

File: ros/src/wojtek_bringup/urdf/wojtek_sim.urdf.xacro (robot description, xacro)
@@ -2,5 +2,5 @@
 <!--
   Visualization/sim URDF: the same mechanics as wojtek_description's
-  four_bar_bot.urdf.xacro (base + imu + 4 legs) but without the ros2_control
+  wojtek.urdf.xacro (base + imu + 4 legs) but without the ros2_control
   and Gazebo blocks. Physics comes from the MuJoCo sim node; this model
   only feeds robot_state_publisher / RViz.
@@ -8,4 +8,4 @@
 <robot name="quadruped" xmlns:xacro="http://www.ros.org/wiki/xacro">
   <xacro:include filename="$(find wojtek_description)/urdf/body.urdf.xacro" />
-  <xacro:four_bar_bot_body />
+  <xacro:wojtek_body />
 </robot>

File: ros/src/wojtek_description/urdf/body.urdf.xacro (robot description, xacro)
@@ -1,4 +1,4 @@
 <?xml version="1.0"?>
-<robot xmlns:xacro="http://www.ros.org/wiki/xacro" name="four_bar_bot_body">
+<robot xmlns:xacro="http://www.ros.org/wiki/xacro" name="wojtek_body">
   <xacro:include filename="$(find wojtek_description)/urdf/inertia.urdf.xacro" />
   <xacro:include filename="$(find wojtek_description)/urdf/leg.urdf.xacro" />
@@ -6,6 +6,6 @@
        base_link/body_link/imu_link, and the four legs. ros2_control/Gazebo
        blocks are deliberately not part of this macro - callers add their
-       own on top (see four_bar_bot.urdf.xacro for the stock example). -->
-  <xacro:macro name="four_bar_bot_body">
+       own on top (see wojtek.urdf.xacro for the stock example). -->
+  <xacro:macro name="wojtek_body">
     <material name="grey">
       <color rgba="0.5 0.5 0.5 1" />

File: ros/src/wojtek_description/urdf/wojtek.urdf.xacro (robot description, xacro)
@@ -10,5 +10,5 @@
   <xacro:arg name="use_hardware" default="True" />
   <xacro:arg name="use_sim" default="False" />
-  <xacro:four_bar_bot_body />
+  <xacro:wojtek_body />
   <xacro:quadruperd_ros2_control use_hardware="$(arg use_hardware)" use_sim="$(arg use_sim)" />
   <!-- <xacro:imu_ros2_control/> -->

Commit message: CAN przez CANdle HAT (SPI@8M): integracja ROS, testy benchowe, nowy IMU I2C
- md80_hardware_interface honoruje `bus` (usb/spi) i nowy param `can_baud`
  (1|2|5|8); robot/real.launch domyślnie bus:=spi can_baud:=8 (napędy
  przeflashowane na 8M). Zweryfikowane na sprzęcie: 12/12 napędów @ 400 Hz
  przez SPI, czysty shutdown. Powrót na dongla: bus:=usb can_baud:=1
  + flash napędów z powrotem na 1M (hw_tests: candle_bus_test baud).
- Serialowe IMU (MCU+CP2102) wycofane: nowy arg use_imu (default false)
  w xacro i launchach -- bez podpiętego sprzętu jego component ros2_control
  ubijał cały ros2_control_node przy configure; springy jest IMU-blind,
  więc jazda bez IMU jest OK do czasu interfejsu I2C.
- candle_bus_test: fix sekwencji zmiany bauda -- po configMd80Can napęd
  od razu słucha na nowym baudzie, więc save do flasha musi iść już nim
  (configCandleBaudrate przed configMd80Save); bez tego zmiana żyła tylko
  w RAM i znikała przy power-cycle'u.
- Test benchowy IMU przepisany pod realny sprzęt: Adafruit 5543
  (LSM6DS3TR-C @ 0x6A + LIS3MDL @ 0x1C) zamiast BMX160, katalog
  bmx160_i2c/ -> imu_i2c/. Oba benche PASS na sprzęcie (CAN soak 300 s
  @ min 357 Hz, IMU: wszystkie kryteria).
- Sprzątanie: osierocone meshe (*_merged.dae, stare STL) -- URDF-y ich
  nie referencują.

Gotcha zapisana w hw_tests/README.md: FDCAN 8M wymaga terminacji 120R
na OBU końcach magistrali (1M wybaczał jej brak, 8M nie).

Co-Authored-By: Claude Fable 5 <noreply@anthropic.com>

File: ros/src/wojtek_bringup/urdf/wojtek_real.urdf.xacro (robot description, xacro)
@@ -17,17 +17,25 @@
   <xacro:arg name="kd" default="1.0" />
   <xacro:arg name="max_torque" default="6.0" />
+  <!-- CAN link to the MD80s: CANdle HAT over SPI by default (drives flashed
+       to 8M). bus:=usb can_baud:=1 falls back to the old USB dongle; only
+       works if the drives are flashed back to 1M. -->
+  <xacro:arg name="bus" default="spi" />
+  <xacro:arg name="can_baud" default="8" />
   <xacro:arg name="usb_port" default="/dev/ttyACM0" />
-  <!-- Loaner BMI160 (no magnetometer) until the real BMX160 is sourced;
-       see bmi160_serial_hardware_interface. Swap back to
-       xacro:wojtek_imu_ros2_control below once the real sensor is back.
-       by-id path instead of /dev/ttyUSBx: the CP2102 drops off the bus on
-       a flaky cable and can re-enumerate under a different number; the
-       by-id symlink always points at the current node (the container mounts
-       the host's /dev, so the symlink stays live). -->
+  <!-- The serial IMU (loaner BMI160 behind an MCU + CP2102 bridge) was retired
+       2026-07-17 in favor of the Adafruit 5543 (LSM6DS3TR-C + LIS3MDL) wired
+       straight to the Pi's I2C1; its ros2_control interface does not exist
+       yet, so use_imu defaults to false and the whole IMU component is left
+       out (with the serial hardware gone, configuring it aborts the entire
+       ros2_control_node). Flip to true only with the CP2102 stack physically
+       reconnected. -->
+  <xacro:arg name="use_imu" default="false" />
   <xacro:arg name="imu_port"
     default="/dev/serial/by-id/usb-Silicon_Labs_CP2102_USB_to_UART_Bridge_Controller_0001-if00-port0" />
   <xacro:wojtek_body />
   <xacro:wojtek_ros2_control kp="$(arg kp)" kd="$(arg kd)" max_torque="$(arg max_torque)"
-    usb_port="$(arg usb_port)" />
-  <xacro:wojtek_bmi160_imu_ros2_control port="$(arg imu_port)" />
+    usb_port="$(arg usb_port)" bus="$(arg bus)" can_baud="$(arg can_baud)" />
+  <xacro:if value="$(arg use_imu)">
+    <xacro:wojtek_bmi160_imu_ros2_control port="$(arg imu_port)" />
+  </xacro:if>
 </robot>

File: ros/src/wojtek_bringup/urdf/wojtek_ros2_control.urdf.xacro (robot description, xacro)
@@ -34,10 +34,16 @@
     </joint>
   </xacro:macro>
-  <xacro:macro name="wojtek_ros2_control" params="kp kd max_torque usb_port">
+  <!-- bus: "spi" = CANdle HAT on the Pi header (device defaults to
+       /dev/spidev0.0 inside the driver), "usb" = the legacy CANdle dongle at
+       usb_port. can_baud (Mbps) must match the drives' flashed baudrate:
+       8 since the 2026-07-17 migration for the HAT; the dongle setup ran 1.
+       See ros/hw_tests/README.md for the per-drive baud migration tool. -->
+  <xacro:macro name="wojtek_ros2_control" params="kp kd max_torque usb_port bus:=spi can_baud:=8">
     <ros2_control name="MD80HardwareInterface" type="system">
       <hardware>
         <plugin>md80_hardware_interface/MD80HardwareInterface</plugin>
         <param name="usb_port">${usb_port}</param>
-        <param name="bus">usb</param>
+        <param name="bus">${bus}</param>
+        <param name="can_baud">${can_baud}</param>
       </hardware>
       <xacro:wojtek_joint name="front_left_first_joint" can_id="10" kp="${kp}" kd="${kd}" max_torque="${max_torque}" />

Commit message: IMU I2C: nowy plugin ros2_control + sprzątanie martwego kodu
Nowa paczka imu_i2c_hardware_interface: SensorInterface dla Adafruit 5543
(LSM6DS3TR-C + LIS3MDL) po I2C, bez pośredniczącego MCU -- rejestrowy
protokół 1:1 z zaliczonego benchu hw_tests/imu_i2c_test.py (raw I2C_RDWR
ioctl, zero dodatkowych zależności). orientation.* eksportowane, ale na
stałe (0,0,0,0): chip nie ma fuzji, a policy_node już ma fallback na
własny filtr komplementarny gdy kwaternion jest zerowy. Błąd I2C w read()
trzyma ostatnią wartość zamiast NaN, configure na złym WHO_AM_I zwraca
ERROR zamiast ubijać cały ros2_control_node. Wpięte jako nowe makro
wojtek_imu_i2c_ros2_control, aktywowane pod use_imu:=true w
wojtek_real.urdf.xacro (imu_port -> imu_bus/imu_addr_ag/imu_addr_mag w
real.launch.py i robot.launch.py); default use_imu nadal false do
pierwszego testu na sprzęcie.

Usunięta martwa gałąź Gazebo z wojtek_description: wojtek.urdf.xacro,
gazebo.urdf.xacro, ros2_control.urdf.xacro oraz trzy launche
(bringup/robot_state_publisher/simulation), których nic nie wołało --
dwa z nich referencjonowały quadruped_controller, którego w tym repo w
ogóle nie ma. Pusty launch/ skasowany, CMakeLists.txt zaktualizowany.

Usunięte martwe makra wojtek_imu_ros2_control (BMX160) i
wojtek_bmi160_imu_ros2_control (BMI160 serial) z
wojtek_ros2_control.urdf.xacro -- nic ich już nie wołało po podmianie
na I2C. Same paczki bmx160_serial_hardware_interface/
bmi160_serial_hardware_interface zostają na razie nietknięte (backlog:
skasować dopiero po teście nowego drivera na robocie).

Co-Authored-By: Claude Sonnet 5 <noreply@anthropic.com>

File: ros/src/wojtek_bringup/urdf/wojtek_real.urdf.xacro (robot description, xacro)
@@ -8,6 +8,6 @@
       was trained against (kp=20, kd=1, +/-6 Nm). Override via xacro args
       for cautious first tests, e.g. max_torque:=2
-    * the BMX160 IMU ros2_control sensor is instantiated (it is commented out
-      in the original description).
+    * the IMU I2C ros2_control sensor is instantiated when use_imu:=true (it
+      is commented out in the original description).
 -->
 <robot name="quadruped" xmlns:xacro="http://www.ros.org/wiki/xacro">
@@ -25,17 +25,17 @@
   <!-- The serial IMU (loaner BMI160 behind an MCU + CP2102 bridge) was retired
        2026-07-17 in favor of the Adafruit 5543 (LSM6DS3TR-C + LIS3MDL) wired
-       straight to the Pi's I2C1; its ros2_control interface does not exist
-       yet, so use_imu defaults to false and the whole IMU component is left
-       out (with the serial hardware gone, configuring it aborts the entire
-       ros2_control_node). Flip to true only with the CP2102 stack physically
-       reconnected. -->
+       straight to the Pi's I2C1: bench-tested (ros/hw_tests/imu_i2c), not
+       yet run through ros2_control on the robot. use_imu still defaults to
+       false until that first hardware test passes. -->
   <xacro:arg name="use_imu" default="false" />
-  <xacro:arg name="imu_port"
-    default="/dev/serial/by-id/usb-Silicon_Labs_CP2102_USB_to_UART_Bridge_Controller_0001-if00-port0" />
+  <xacro:arg name="imu_bus" default="/dev/i2c-1" />
+  <xacro:arg name="imu_addr_ag" default="0x6A" />
+  <xacro:arg name="imu_addr_mag" default="0x1C" />
   <xacro:wojtek_body />
   <xacro:wojtek_ros2_control kp="$(arg kp)" kd="$(arg kd)" max_torque="$(arg max_torque)"
     usb_port="$(arg usb_port)" bus="$(arg bus)" can_baud="$(arg can_baud)" />
   <xacro:if value="$(arg use_imu)">
-    <xacro:wojtek_bmi160_imu_ros2_control port="$(arg imu_port)" />
+    <xacro:wojtek_imu_i2c_ros2_control bus="$(arg imu_bus)" addr_ag="$(arg imu_addr_ag)"
+      addr_mag="$(arg imu_addr_mag)" />
   </xacro:if>
 </robot>

File: ros/src/wojtek_bringup/urdf/wojtek_ros2_control.urdf.xacro (robot description, xacro)
@@ -61,12 +61,19 @@
     </ros2_control>
   </xacro:macro>
-  <!-- baud_rate must match the firmware's Serial.begin(), i.e. 115200 in
-       bmx160_serial_hardware_interface/firmware/main/main.ino. -->
-  <xacro:macro name="wojtek_imu_ros2_control" params="port baud_rate:=115200">
+  <!-- Adafruit 5543 (LSM6DS3TR-C + LIS3MDL) straight on the Pi's I2C bus:
+       no MCU/firmware bridge, no onboard fusion. orientation.* is exported
+       (imu_sensor_broadcaster requires it) but the driver always writes
+       (0,0,0,0); wojtek_policy's IMU callback treats that as "no fusion"
+       and runs its own accel+gyro complementary filter instead. addr_ag/
+       addr_mag default to the board's un-jumpered addresses; bump to
+       0x6B/0x1E if SDO is pulled high. See ros/hw_tests/imu_i2c for the
+       bench test this register map/init sequence was validated against. -->
+  <xacro:macro name="wojtek_imu_i2c_ros2_control" params="bus:=/dev/i2c-1 addr_ag:=0x6A addr_mag:=0x1C">
     <ros2_control name="imu" type="sensor">
       <hardware>
-        <plugin>bmx160_serial_hardware_interface/BMX160SerialHardwareInterface</plugin>
-        <param name="port">${port}</param>
-        <param name="baud_rate">${baud_rate}</param>
+        <plugin>imu_i2c_hardware_interface/ImuI2CHardwareInterface</plugin>
+        <param name="bus">${bus}</param>
+        <param name="addr_ag">${addr_ag}</param>
+        <param name="addr_mag">${addr_mag}</param>
       </hardware>
       <sensor name="imu">
@@ -87,29 +94,3 @@
     </ros2_control>
   </xacro:macro>
-  <!-- Loaner sensor stand-in for wojtek_imu_ros2_control above: a bare BMI160
-       (accel+gyro only, no magnetometer) is what's actually wired in until
-       a real BMX160 is sourced. See bmi160_serial_hardware_interface for
-       why magnetometer.* is dropped: nothing downstream (imu_sensor_broadcaster,
-       wojtek_policy) consumes it anyway. -->
-  <xacro:macro name="wojtek_bmi160_imu_ros2_control" params="port baud_rate:=115200">
-    <ros2_control name="imu" type="sensor">
-      <hardware>
-        <plugin>bmi160_serial_hardware_interface/BMI160SerialHardwareInterface</plugin>
-        <param name="port">${port}</param>
-        <param name="baud_rate">${baud_rate}</param>
-      </hardware>
-      <sensor name="imu">
-        <state_interface name="orientation.x" />
-        <state_interface name="orientation.y" />
-        <state_interface name="orientation.z" />
-        <state_interface name="orientation.w" />
-        <state_interface name="angular_velocity.x" />
-        <state_interface name="angular_velocity.y" />
-        <state_interface name="angular_velocity.z" />
-        <state_interface name="linear_acceleration.x" />
-        <state_interface name="linear_acceleration.y" />
-        <state_interface name="linear_acceleration.z" />
-      </sensor>
-    </ros2_control>
-  </xacro:macro>
 </robot>
