Commit message: feat(deploy): carry the tau_ff head end-to-end from export to the MD80 drives
The schema-2 contract now classifies task.env.tau_ff and ships a "tau_ff"
block (enable + scale); the whole chain applies it:

- wojtek_policy runtime: 24-wide MLP output, filter over the full action,
  targets from the position half (obs last_act stays 12-wide as trained),
  torque half exposed as last_tau_ff = clip(scale*act[12:], +-scale).
  Export validates the runtime torque against the env reference in
  normalized units (the N*m compare would scale float32 matmul noise by
  tau_ff.scale past the radians-calibrated bound).
- policy_node publishes the torque as JointState.effort on
  /wojtek/joint_targets (URDF sign convention, soft-start gated).
- real_io_node forwards it to forward_effort_controller/commands (no boot
  offset -- torque is frame-free) and drops the WHOLE command on a
  non-finite effort.
- md80_hardware_interface accepts a [position, effort] interface pair in
  IMPEDANCE mode and writes setTargetTorque (the drive's native
  tau = kp*e - kd*dq + tau_ff), non-finite guarded to 0.
- launch_common reads the head from the loaded contract (a tau_ff policy
  stays a config change): tau_ff:=true to the xacro (per-joint effort
  command interface), forward_effort_controller spawned, and the DRIVE
  torque limit widened to pd.max_torque + tau_ff.scale -- the sim clamps
  servo and head separately, the drive clamps the sum, so the widened cap
  is the superset match.
- mujoco_sim_node applies the same effort as qfrc_applied for sim parity.

Validated: export of wojtek_flat_tff_sag_v2b_s0 round-trips at 3.7e-5
(numpy vs brax bitwise) with action_size 24 + tau_ff{enable,scale:3};
legacy 12-action keeper export unchanged (9.4e-7, head disabled); 28
wojtek_policy unit tests incl. new head coverage; 431 training unit
tests. verify-static's two failures reproduce on a clean tree
(pre-existing baseline drift). The C++ change compiles only in the ROS
gate; run make verify before robot use.

Co-Authored-By: Claude Fable 5 <noreply@anthropic.com>

File: ros/src/wojtek_bringup/urdf/wojtek_real.urdf.xacro (robot description, xacro)
@@ -18,4 +18,9 @@
   <xacro:arg name="kd" default="1.6" />
   <xacro:arg name="max_torque" default="9.0" />
+  <!-- Feed-forward torque head (tau_ff policies): exposes an `effort`
+       command interface per joint on top of `position`. The launch sets it
+       from the loaded policy's contract and widens max_torque to
+       pd.max_torque + tau_ff.scale (the sim clamps the two separately). -->
+  <xacro:arg name="tau_ff" default="false" />
   <!-- CAN link to the MD80s: CANdle HAT over SPI by default (drives flashed
        to 8M). bus:=usb can_baud:=1 falls back to the old USB dongle; only
@@ -38,5 +43,5 @@
   <xacro:wojtek_ros2_control kp="$(arg kp)" kd="$(arg kd)" max_torque="$(arg max_torque)"
     usb_port="$(arg usb_port)" bus="$(arg bus)" can_baud="$(arg can_baud)"
-    dry_run="$(arg dry_run)" />
+    dry_run="$(arg dry_run)" tau_ff="$(arg tau_ff)" />
   <xacro:if value="$(arg use_imu)">
     <xacro:wojtek_imu_i2c_ros2_control bus="$(arg imu_bus)" addr_ag="$(arg imu_addr_ag)"

File: ros/src/wojtek_bringup/urdf/wojtek_ros2_control.urdf.xacro (robot description, xacro)
@@ -5,8 +5,19 @@
        exactly the actuator model the policy was trained with
        (wojtek_mjx.xml: gainprm=20, biasprm="0 -20 -1", forcerange 6)
-       when kp=20, kd=1, max_torque=6. -->
-  <xacro:macro name="wojtek_joint" params="name can_id kp kd max_torque">
+       when kp=20, kd=1, max_torque=6.
+       tau_ff=true (wired from the loaded policy's contract) additionally
+       exposes an `effort` command interface on every joint: impedance-mode
+       feed-forward torque, added by the drive ON TOP of the PD law
+       (tau = kp*e - kd*dq + tau_ff). The training sim clamps the servo
+       (max_torque) and the head (tau_ff.scale) separately, so pass a
+       max_torque that covers their SUM (launch does: pd.max_torque +
+       tau_ff.scale); a tighter drive cap would truncate the trained
+       torque envelope. -->
+  <xacro:macro name="wojtek_joint" params="name can_id kp kd max_torque tau_ff:=false">
     <joint name="${name}">
       <command_interface name="position" />
+      <xacro:if value="${tau_ff}">
+        <command_interface name="effort" />
+      </xacro:if>
       <state_interface name="position">
         <param name="initial_value">0.0</param>
@@ -39,5 +50,5 @@
        8 since the 2026-07-17 migration for the HAT; the dongle setup ran 1.
        See ros/hw_tests/README.md for the per-drive baud migration tool. -->
-  <xacro:macro name="wojtek_ros2_control" params="kp kd max_torque usb_port bus:=spi can_baud:=8 dry_run:=false">
+  <xacro:macro name="wojtek_ros2_control" params="kp kd max_torque usb_port bus:=spi can_baud:=8 dry_run:=false tau_ff:=false">
     <ros2_control name="MD80HardwareInterface" type="system">
       <hardware>
@@ -50,16 +61,16 @@
         <param name="dry_run">${dry_run}</param>
       </hardware>
-      <xacro:wojtek_joint name="front_left_first_joint" can_id="10" kp="${kp}" kd="${kd}" max_torque="${max_torque}" />
-      <xacro:wojtek_joint name="front_left_second_joint" can_id="11" kp="${kp}" kd="${kd}" max_torque="${max_torque}" />
-      <xacro:wojtek_joint name="front_left_third_joint" can_id="12" kp="${kp}" kd="${kd}" max_torque="${max_torque}" />
-      <xacro:wojtek_joint name="front_right_first_joint" can_id="20" kp="${kp}" kd="${kd}" max_torque="${max_torque}" />
-      <xacro:wojtek_joint name="front_right_second_joint" can_id="21" kp="${kp}" kd="${kd}" max_torque="${max_torque}" />
-      <xacro:wojtek_joint name="front_right_third_joint" can_id="22" kp="${kp}" kd="${kd}" max_torque="${max_torque}" />
-      <xacro:wojtek_joint name="rear_right_first_joint" can_id="30" kp="${kp}" kd="${kd}" max_torque="${max_torque}" />
-      <xacro:wojtek_joint name="rear_right_second_joint" can_id="31" kp="${kp}" kd="${kd}" max_torque="${max_torque}" />
-      <xacro:wojtek_joint name="rear_right_third_joint" can_id="32" kp="${kp}" kd="${kd}" max_torque="${max_torque}" />
-      <xacro:wojtek_joint name="rear_left_first_joint" can_id="40" kp="${kp}" kd="${kd}" max_torque="${max_torque}" />
-      <xacro:wojtek_joint name="rear_left_second_joint" can_id="41" kp="${kp}" kd="${kd}" max_torque="${max_torque}" />
-      <xacro:wojtek_joint name="rear_left_third_joint" can_id="42" kp="${kp}" kd="${kd}" max_torque="${max_torque}" />
+      <xacro:wojtek_joint name="front_left_first_joint" can_id="10" kp="${kp}" kd="${kd}" max_torque="${max_torque}" tau_ff="${tau_ff}" />
+      <xacro:wojtek_joint name="front_left_second_joint" can_id="11" kp="${kp}" kd="${kd}" max_torque="${max_torque}" tau_ff="${tau_ff}" />
+      <xacro:wojtek_joint name="front_left_third_joint" can_id="12" kp="${kp}" kd="${kd}" max_torque="${max_torque}" tau_ff="${tau_ff}" />
+      <xacro:wojtek_joint name="front_right_first_joint" can_id="20" kp="${kp}" kd="${kd}" max_torque="${max_torque}" tau_ff="${tau_ff}" />
+      <xacro:wojtek_joint name="front_right_second_joint" can_id="21" kp="${kp}" kd="${kd}" max_torque="${max_torque}" tau_ff="${tau_ff}" />
+      <xacro:wojtek_joint name="front_right_third_joint" can_id="22" kp="${kp}" kd="${kd}" max_torque="${max_torque}" tau_ff="${tau_ff}" />
+      <xacro:wojtek_joint name="rear_right_first_joint" can_id="30" kp="${kp}" kd="${kd}" max_torque="${max_torque}" tau_ff="${tau_ff}" />
+      <xacro:wojtek_joint name="rear_right_second_joint" can_id="31" kp="${kp}" kd="${kd}" max_torque="${max_torque}" tau_ff="${tau_ff}" />
+      <xacro:wojtek_joint name="rear_right_third_joint" can_id="32" kp="${kp}" kd="${kd}" max_torque="${max_torque}" tau_ff="${tau_ff}" />
+      <xacro:wojtek_joint name="rear_left_first_joint" can_id="40" kp="${kp}" kd="${kd}" max_torque="${max_torque}" tau_ff="${tau_ff}" />
+      <xacro:wojtek_joint name="rear_left_second_joint" can_id="41" kp="${kp}" kd="${kd}" max_torque="${max_torque}" tau_ff="${tau_ff}" />
+      <xacro:wojtek_joint name="rear_left_third_joint" can_id="42" kp="${kp}" kd="${kd}" max_torque="${max_torque}" tau_ff="${tau_ff}" />
     </ros2_control>
   </xacro:macro>
