Commit message: fix(imu): pass a speed_t constant to cfsetospeed, not the bit rate
The IMU was silent on the real robot: ros2_control logged "incomplete IMU
read" every second and policy_node correctly held with "non-finite sensor
input", so no targets were ever published.

cfsetospeed/cfsetispeed expect a speed_t constant (B115200 == 4098), not the
literal 115200 the URDF carries. Called with the bit rate they return -1/EINVAL
and leave c_cflag untouched -- and both return values were ignored, so the port
stayed at its 9600 default while the firmware streamed at 115200. The reader saw
only noise, every field stayed NaN.

Confirmed on hardware: `stty -F /dev/ttyUSB0` reported 9600; reading the port at
115200 yields well-formed frames ("R X: 0.01 Y: 0.02 Z: 0.23 W: 0.97"), at 9600
nothing. The sensor was fine all along.

Map the integer onto the constant and fail loudly on an unsupported rate or a
cfset* error. The same copied code was broken in both IMU packages.

Also bring the BMX160 macro's baud default to 115200: it declared 9600 while its
firmware runs at 115200 -- harmless while the rate never applied, but this fix
would have made 9600 take effect and silence that sensor for real.

Also install setserial on the RPi. CANdle shells out to `setserial <port>
low_latency` and fell back to "low-speed mode" without it, adding latency to the
400 Hz loop. The PC image already had it; the RPi, where it matters, did not.

Co-Authored-By: Claude Opus 4.8 <noreply@anthropic.com>

File: ros/src/wojtek_bringup/urdf/wojtek_ros2_control.urdf.xacro (robot description, xacro)
@@ -55,5 +55,7 @@
     </ros2_control>
   </xacro:macro>
-  <xacro:macro name="wojtek_imu_ros2_control" params="port baud_rate:=9600">
+  <!-- baud_rate must match the firmware's Serial.begin(), i.e. 115200 in
+       bmx160_serial_hardware_interface/firmware/main/main.ino. -->
+  <xacro:macro name="wojtek_imu_ros2_control" params="port baud_rate:=115200">
     <ros2_control name="imu" type="sensor">
       <hardware>

Commit message: feat(imu): 9-DoF fusion -- mag on a topic + orientation ESKF in the driver
The Adafruit 5543 pair (LSM6DS3TR-C + LIS3MDL) has no onboard fusion, so
orientation.* was pinned to (0,0,0,0) and wojtek_policy fell back to its
accel+gyro complementary filter; the magnetometer never reached a topic
at all (upstream imu_sensor_broadcaster ignores magnetometer.*).

* magnetometer_broadcaster (new package): minimal ros2_control broadcaster
  publishing magnetometer.{x,y,z} as sensor_msgs/MagneticField on
  ~/magnetic_field; wired into real_controllers.yaml and both launches,
  declared as a wojtek_bringup dep so deploy's --packages-up-to builds it
  on the RPi (its absence killed the spawner on first hardware try).

* orientation ESKF in imu_i2c_hardware_interface: error-state KF
  (quaternion + gyro bias, Sola conventions) -- gyro predicts, accel
  corrects roll/pitch, mag corrects YAW ONLY so drive-current field
  disturbance cannot leak into the gravity vector the policy consumes.
  Mag R adapts with |B|-vs-norm deviation and innovation (Mahalanobis
  gate drops gross outliers): during motor transients the filter rides
  the gyro, and the continuously estimated bias keeps that drift slow --
  aimed squarely at the yaw drift seen on the first walk. orientation.*
  stays (0,0,0,0) until the first accel+mag init, which policy_node
  already treats as "no fusion yet" (rollback: gravity_from_accel).
  Covered by 7 gtests on synthetic data (init, bias convergence, yaw
  tracking, disturbance gating, mag-outage recovery, hard-iron).

* driver reads STATUS_REG data-ready and merges status+data into one
  I2C burst per chip (16 B + 7 B): the 400 Hz read() budget is 2.5 ms
  and separate status transactions pushed it to 3.3 ms (overruns on
  hardware). install.sh now also provisions i2c_arm_baudrate=400000
  (both chips do Fast Mode) taking the burst from ~2.3 ms to ~0.6 ms.

* mag_calib.py (hw_tests/imu_i2c): drone-style ellipsoid calibration --
  rotate the robot, fit hard/soft iron + field norm, write the yaml the
  driver loads via the new mag_calib_file param (identity placeholder
  ships in wojtek_bringup/config/mag_calib.yaml). Rejects fits with
  poor octant coverage; validated on synthetic distorted data.

Co-Authored-By: Claude Opus 4.8 <noreply@anthropic.com>

File: ros/src/wojtek_bringup/urdf/wojtek_ros2_control.urdf.xacro (robot description, xacro)
@@ -65,12 +65,16 @@
   </xacro:macro>
   <!-- Adafruit 5543 (LSM6DS3TR-C + LIS3MDL) straight on the Pi's I2C bus:
-       no MCU/firmware bridge, no onboard fusion. orientation.* is exported
-       (imu_sensor_broadcaster requires it) but the driver always writes
-       (0,0,0,0); wojtek_policy's IMU callback treats that as "no fusion"
-       and runs its own accel+gyro complementary filter instead. addr_ag/
-       addr_mag default to the board's un-jumpered addresses; bump to
-       0x6B/0x1E if SDO is pulled high. See ros/hw_tests/imu_i2c for the
+       no MCU/firmware bridge, no onboard fusion. orientation.* carries the
+       quaternion from the driver's error-state Kalman filter (gyro
+       prediction + accel roll/pitch + mag yaw, orientation_eskf.hpp); it
+       reads (0,0,0,0) only until the filter sees its first accel+mag pair,
+       which wojtek_policy treats as "no fusion yet" and bridges with its
+       own complementary filter. mag_calib_file points at the ellipsoid
+       calibration produced by ros/hw_tests/imu_i2c/mag_calib.py (the
+       shipped default is an identity placeholder; usable, uncalibrated).
+       addr_ag/addr_mag default to the board's un-jumpered addresses; bump
+       to 0x6B/0x1E if SDO is pulled high. See ros/hw_tests/imu_i2c for the
        bench test this register map/init sequence was validated against. -->
-  <xacro:macro name="wojtek_imu_i2c_ros2_control" params="bus:=/dev/i2c-1 addr_ag:=0x6A addr_mag:=0x1C">
+  <xacro:macro name="wojtek_imu_i2c_ros2_control" params="bus:=/dev/i2c-1 addr_ag:=0x6A addr_mag:=0x1C mag_calib_file:='$(find wojtek_bringup)/config/mag_calib.yaml'">
     <ros2_control name="imu" type="sensor">
       <hardware>
@@ -79,4 +83,5 @@
         <param name="addr_ag">${addr_ag}</param>
         <param name="addr_mag">${addr_mag}</param>
+        <param name="mag_calib_file">${mag_calib_file}</param>
       </hardware>
       <sensor name="imu">

Commit message: config(ros): drives flashed to 1M -- make can_baud:=1 the default
The twelve MD80s run at 1M again (ros/hw_tests candle_bus_test baud, flash
saved); the launch and xacro defaults now say so, with the reason: on this
harness the termination lives only in the two CANdles at the bus ends, so
every in-line connector carries the far terminator and 8M lost frames,
flash writes and -- on a lost terminator -- all twelve drives at once. At
1M the same harness holds under plug movement. The hw_tests README keeps
the 8M procedure for a fixed harness and records the retry quirk of flash
saves at 8M.

Co-Authored-By: Claude Fable 5.1 <noreply@anthropic.com>

File: ros/src/wojtek_bringup/urdf/wojtek_ros2_control.urdf.xacro (robot description, xacro)
@@ -48,7 +48,8 @@
        /dev/spidev0.0 inside the driver), "usb" = the legacy CANdle dongle at
        usb_port. can_baud (Mbps) must match the drives' flashed baudrate:
-       8 since the 2026-07-17 migration for the HAT; the dongle setup ran 1.
-       See ros/hw_tests/README.md for the per-drive baud migration tool. -->
-  <xacro:macro name="wojtek_ros2_control" params="kp kd max_torque usb_port bus:=spi can_baud:=8 dry_run:=false tau_ff:=false">
+       1 since 2026-10-05 (8 from the 2026-07-17 HAT migration until then;
+       the harness could not hold 8M -- see launch_common.py). The launch
+       passes it; see ros/hw_tests/README.md for the per-drive baud tool. -->
+  <xacro:macro name="wojtek_ros2_control" params="kp kd max_torque usb_port bus:=spi can_baud:=1 dry_run:=false tau_ff:=false">
     <ros2_control name="MD80HardwareInterface" type="system">
       <hardware>
