Commit message: salvage: the robot's ~/wojtek_ws/src tree as found on the RPi on 2026-10-23
Snapshot of the robot's workspace (not a git repo on the RPi) before the
first deploy of the new-legs stack. ros/src is the RPi tree verbatim minus
wojtek_pc (never on the robot); ros/deploy/rpi/robot-local holds the
systemd drop-in and the on-robot scripts.

Co-Authored-By: Claude Fable 5.1 <noreply@anthropic.com>

File: ros/src/wojtek_bringup/urdf/wojtek_mock_ros2_control.urdf.xacro (robot description, xacro)
@@ -60,7 +60,9 @@
       <xacro:wojtek_mock_joint name="rear_left_second_joint" tau_ff="${tau_ff}" />
       <xacro:wojtek_mock_joint name="rear_left_third_joint" tau_ff="${tau_ff}" />
-      <!-- A level, motionless robot with the sensor upright (URDF imu_joint
-           rpy 0 0 0): identity orientation, +g on the accelerometer's z. The
-           policy only needs finite, fresh values to run its full tick. -->
+      <!-- A level, motionless robot with the sensor upright: identity
+           orientation, +g on the accelerometer's z. URDF imu_joint only
+           yaws the sensor, which changes neither, so identity is a valid
+           level reading. The policy only needs finite, fresh values to run
+           its full tick. -->
       <xacro:if value="${use_imu}">
         <sensor name="imu">

File: ros/src/wojtek_bringup/urdf/wojtek_real.urdf.xacro (robot description, xacro)
@@ -49,5 +49,11 @@
        See wojtek_mock_ros2_control.urdf.xacro. -->
   <xacro:arg name="mock_hw" default="false" />
-  <xacro:wojtek_body />
+  <!-- with_camera_mount: the D435's mount (base_link -> camera_link) and
+       nothing below it. The driver publishes camera_link -> *_optical
+       itself; the mount is the one edge it cannot know, and here the
+       robot_state_publisher gives it in every mode that runs a camera
+       (deck_camera:=true, perception:=true), which the costmap, the pixel
+       resolver and the VLM brain's bearing all need. -->
+  <xacro:wojtek_body with_camera_mount="true" />
   <xacro:if value="$(arg mock_hw)">
     <xacro:wojtek_mock_ros2_control use_imu="$(arg use_imu)" tau_ff="$(arg tau_ff)" />

File: ros/src/wojtek_description/urdf/body.urdf.xacro (robot description, xacro)
@@ -7,12 +7,40 @@
        blocks are deliberately not part of this macro - callers add their
        own on top (see wojtek.urdf.xacro for the stock example).
-       with_camera adds the D435 mount frames (camera_link + optical
-       frames). Default OFF: on the real robot the realsense2_camera driver
-       publishes the camera_link->*_optical chain itself and two publishers
-       of the same TF edge fight. The sim URDF turns it on: there the
-       robot model owns the ground-truth extrinsics (machinekind/wojtek#91).
+       The D435 comes in two shapes, both default OFF, never both on:
+         with_camera_mount  base_link -> camera_link only. The real robot:
+                            the realsense2_camera driver publishes the
+                            camera_link -> *_optical chain itself (two
+                            publishers of one TF edge fight), but cannot
+                            know where the camera sits on the body, and the
+                            costmap, the pixel resolver and the VLM brain
+                            need that edge in every mode with a camera.
+         with_camera        the mount and the optical frames. The sim: the
+                            robot model owns the ground-truth extrinsics
+                            (machinekind/wojtek#91).
        The mount numbers must match wojtek_pc/camera_spec.py (MOUNT_XYZ,
-       MOUNT_PITCH_RAD); a test cross-checks them. -->
-  <xacro:macro name="wojtek_body" params="with_camera:=false">
+       MOUNT_PITCH_RAD) and wojtek_perception_bringup/config/extrinsics.yaml;
+       tests cross-check all three. -->
+  <xacro:macro name="camera_mount">
+    <!-- D435 mount: camera_link (x forward, z up, ROS body convention)
+         at the centre of the head bracket (front face of the body mesh's
+         triangular head section), pitched 15 deg down (0.2617994 rad). -->
+    <link name="camera_link">
+      <visual>
+        <!-- Camera-body sized marker so the mount is visible in RViz;
+             massless. -->
+        <origin xyz="-0.01 0 0" rpy="0 0 0" />
+        <geometry>
+          <box size="0.02 0.09 0.025" />
+        </geometry>
+        <xacro:grey_material />
+      </visual>
+    </link>
+    <joint name="camera_joint" type="fixed">
+      <parent link="base_link" />
+      <child link="camera_link" />
+      <origin xyz="0.32 0.0 0.07" rpy="0 0.2617994 0" />
+    </joint>
+  </xacro:macro>
+  <xacro:macro name="wojtek_body" params="with_camera:=false with_camera_mount:=false">
     <material name="grey">
       <color rgba="0.5 0.5 0.5 1" />
@@ -41,8 +69,12 @@
     </joint>
     <link name="imu_link" />
-    <!-- The Adafruit 5543 sits UPRIGHT: measured at rest on the robot,
-         linear_acceleration.z = +10.05 m/s2, and imu_i2c.cpp reads the chip
-         axes straight into x/y/z with no remap. The rpy 0 pi 0 that stood
-         here was left over from the previous IMU and made policy_node flip
+    <!-- The Adafruit 5543 sits UPRIGHT (measured at rest on the robot,
+         linear_acceleration.z = +10.05 m/s2) and yawed -90 deg: the chip's
+         +y points forward, its +x to the robot's right. imu_i2c.cpp reads
+         the chip axes straight into x/y/z with no remap, so this rotation
+         is the only place the mount is undone; launch_common's
+         IMU_MOUNT_RPY copies it for policy_node and leg_odometry, and
+         wojtek_sim.urdf.xacro's imu_mount_rpy emulates it. An earlier
+         rpy 0 pi 0 left over from the previous IMU made policy_node flip
          gravity and the gyro's x/z, which stayed invisible until a policy
          actually read the IMU (terrain_blind v41). That one then fought a
@@ -51,31 +83,15 @@
       <parent link="base_link" />
       <child link="imu_link" />
-      <origin xyz="0.0 0.0 0.1" rpy="0.0 0.0 0.0" />
+      <origin xyz="0.053 0.0 0.012" rpy="0.0 0.0 -1.5707963" />
     </joint>
+    <xacro:if value="${with_camera_mount}">
+      <xacro:camera_mount />
+    </xacro:if>
     <xacro:if value="${with_camera}">
-      <!-- D435 mount: camera_link (x forward, z up, ROS body convention)
-           at the centre of the head bracket (front face of the body mesh's
-           triangular head section), pitched down; then the standard
-           camera_frame -> optical_frame (z forward, x right, y down)
-           rotation. Frame names follow the realsense2_camera driver
-           (camera_name=camera) so consumers see identical TF in sim and
-           on the robot. Values mirror camera_spec.py: MOUNT_XYZ /
-           MOUNT_PITCH_RAD (15 deg = 0.2617994 rad). -->
-      <link name="camera_link">
-        <visual>
-          <!-- Camera-body sized marker so the mount is visible in RViz;
-               massless. -->
-          <origin xyz="-0.01 0 0" rpy="0 0 0" />
-          <geometry>
-            <box size="0.02 0.09 0.025" />
-          </geometry>
-          <xacro:grey_material />
-        </visual>
-      </link>
-      <joint name="camera_joint" type="fixed">
-        <parent link="base_link" />
-        <child link="camera_link" />
-        <origin xyz="0.32 0.0 0.07" rpy="0 0.2617994 0" />
-      </joint>
+      <!-- The mount, then the standard camera_frame -> optical_frame
+           (z forward, x right, y down) rotation. Frame names follow the
+           realsense2_camera driver (camera_name=camera) so consumers see
+           identical TF in sim and on the robot. -->
+      <xacro:camera_mount />
       <link name="camera_depth_frame" />
       <joint name="camera_depth_joint" type="fixed">
