Commit message: feat(sim): D435-compatible virtual camera in MuJoCo sim (#97)
* feat(sim): D435-compatible virtual camera in MuJoCo sim

Closes the sim/robot perception gap (#91): mujoco_sim_node renders an
offscreen depth + colour camera and publishes it in exactly the format and
on exactly the topics of the real D435 stack, so cloud_reduce, the planner
and (later) the VLM run unchanged against the simulator.

- wojtek_viz/camera_spec.py: single source of truth for the camera
  contract -- 424x240 16UC1 depth in mm (fx=fy=209, ~90 deg HFOV), rgb8
  colour, frame names, topics, the base_link mount pose. FOVY is derived
  from fy so the MJCF camera and CameraInfo cannot drift apart. Depth
  outside 0.3-3.0 m (incl. the renderer's far-plane sky value) becomes 0,
  the RealSense no-return convention.
- wojtek_viz/depth_camera.py: SimDepthCamera owns the offscreen renderers
  and a private MjData; the camera is injected into the sim model at load
  time via MjSpec, keeping this change physics-neutral (the stale model
  copy question is #93). Optional per-call snapshot sync via mj_forward.
- mujoco_sim_node: guarded MUJOCO_GL import (a missing EGL degrades to
  camera-off instead of killing physics), a lock-protected (stamp, qpos,
  qvel) snapshot taken in _tick, and a dedicated render thread that owns
  every GL object (contexts are thread-affine). Image stamps equal the
  odom->base_link TF stamp of the snapshotted physics tick, so tf2
  lookups at image time are exact. New /sim/rtf telemetry plus a catch-up
  cap warning make the real-time-factor criterion measurable.
- URDF: base_link->camera_link->optical frames behind a with_camera macro
  arg (default off; the real D435 driver publishes its own optical chain).
  The sim URDF enables it -- TF comes from the robot model, not a config.
- launch/CLI: camera:=true/false (default on) plus rate args on
  sim.launch.py; robot.py now forwards name:=value tokens (strictly
  validated) so ./sim.sh camera:=false works with no bespoke flag.
- docker: mesa EGL/OSMesa runtime libs for headless offscreen rendering.
- perception.rviz ported from jakuc/perception-d435-bringup for viewing.

* test(sim): camera contract, renderer and URDF-consistency suites

- test_camera_spec.py: intrinsics/FOV algebra, CameraInfo layout,
  depth_to_mm windowing (no ROS, no GL -- runs anywhere).
- test_depth_camera.py: real offscreen renders (skip cleanly without a GL
  backend): encoding/resolution/units, wall-at-known-distance within 1 cm
  with the expectation computed from the model's own cam_xpos/cam_xmat
  (the renders-from-head-pose criterion at unit level), sky/no-return = 0,
  out-of-window clipping, and the camera following a moved base.
- test_camera_model_consistency.py: URDF camera frames vs camera_spec vs
  the MJCF injection -- catches the camera-moved-but-TF-stale bug class.

* docs: virtual D435 camera in the ROS architecture reference

mujoco_sim_node topic table, camera parameters, sim data-flow diagram
(cloud_reduce fed by the virtual camera) and sim.launch.py arguments.

* fix(docker): NVIDIA GPU passthrough so the container renders on hardware

On a host with the proprietary NVIDIA driver the container's mesa cannot
drive the GPU (no userspace driver inside), so RViz and the camera's
offscreen renderer fell back to llvmpipe -- everything painted on the CPU
and a ./sim.sh session was barely responsive, while the same stack ran
fine natively.

compose.gpu.yaml layers runtime:nvidia + NVIDIA_VISIBLE_DEVICES/
NVIDIA_DRIVER_CAPABILITIES on the service; sim.sh and dev.sh include it
only when docker reports the nvidia runtime (nvidia-container-toolkit
installed and registered), so machines without the toolkit keep the
current behaviour. Measured on an RTX 3050 laptop: depth render
10.8 Hz -> 15.0 Hz (frame jitter 47 ms -> 3 ms), RViz GLX renderer
llvmpipe -> NVIDIA, physics RTF 1.00.

Host prerequisite (one-time, documented in compose.gpu.yaml): install
nvidia-container-toolkit, register the runtime, restart docker; on hosts
where the RPM scriptlet fails to generate the CDI spec, run
  sudo nvidia-ctk cdi generate --output=/etc/cdi/nvidia.yaml
and restart docker again.

* feat(viz): sim brings up RViz with the camera panels by default

New wojtek_viz config/sim.rviz = the plain wojtek.rviz view plus the
virtual D435's colour and depth Image panels (Best Effort, matching the
sim's sensor-data QoS), so ./sim.sh shows what the camera sees without
any manual panel-adding. viz.launch.py and sim.launch.py gain an
rviz_config argument (default unchanged for the live robot); robot.py
--sim passes the sim layout.

* feat(sim): move the camera to the head bracket

Mount goes from the placeholder mast (0.18, 0, 0.25) to the centre of the
head bracket -- the front face of the body mesh's triangular head section,
measured from base_link.dae vertices: tip x=0.292, centred y=0, z~0.067.
MOUNT_XYZ = (0.29, 0, 0.07), pitch unchanged at 15 deg down. The RViz
marker becomes a camera-body-sized box instead of the mast.

The camera now sits ~0.2 m over the floor, which puts the floor inside
the valid window on the principal ray, so the wall tests probe a pixel
above the principal point (ray slightly over horizontal -- it can only
hit the wall) and predict depth with the full per-pixel ray formula from
the model's own cam_xpos/cam_xmat.

* feat(sim): nudge the camera 3 cm proud of the head bracket

Lens at x=0.32 (bracket tip is 0.292) so the bracket's edges cannot clip
into the frame; z and the 15 deg pitch unchanged.

---------

Co-authored-by: Greg <user@HOST>

File: ros/src/wojtek_description/urdf/body.urdf.xacro (robot description, xacro)
@@ -6,6 +6,13 @@
        base_link/body_link/imu_link, and the four legs. ros2_control/Gazebo
        blocks are deliberately not part of this macro - callers add their
-       own on top (see wojtek.urdf.xacro for the stock example). -->
-  <xacro:macro name="wojtek_body">
+       own on top (see wojtek.urdf.xacro for the stock example).
+       with_camera adds the D435 mount frames (camera_link + optical
+       frames). Default OFF: on the real robot the realsense2_camera driver
+       publishes the camera_link->*_optical chain itself and two publishers
+       of the same TF edge fight. The sim URDF turns it on: there the
+       robot model owns the ground-truth extrinsics (machinekind/wojtek#91).
+       The mount numbers must match wojtek_viz/camera_spec.py (MOUNT_XYZ,
+       MOUNT_PITCH_RAD); a test cross-checks them. -->
+  <xacro:macro name="wojtek_body" params="with_camera:=false">
     <material name="grey">
       <color rgba="0.5 0.5 0.5 1" />
@@ -39,4 +46,54 @@
       <origin xyz="0.0 0.0 0.1" rpy=" 0.0 ${pi} 0.0" />
     </joint>
+    <xacro:if value="${with_camera}">
+      <!-- D435 mount: camera_link (x forward, z up, ROS body convention)
+           at the centre of the head bracket (front face of the body mesh's
+           triangular head section), pitched down; then the standard
+           camera_frame -> optical_frame (z forward, x right, y down)
+           rotation. Frame names follow the realsense2_camera driver
+           (camera_name=camera) so consumers see identical TF in sim and
+           on the robot. Values mirror camera_spec.py: MOUNT_XYZ /
+           MOUNT_PITCH_RAD (15 deg = 0.2617994 rad). -->
+      <link name="camera_link">
+        <visual>
+          <!-- Camera-body sized marker so the mount is visible in RViz;
+               massless. -->
+          <origin xyz="-0.01 0 0" rpy="0 0 0" />
+          <geometry>
+            <box size="0.02 0.09 0.025" />
+          </geometry>
+          <xacro:grey_material />
+        </visual>
+      </link>
+      <joint name="camera_joint" type="fixed">
+        <parent link="base_link" />
+        <child link="camera_link" />
+        <origin xyz="0.32 0.0 0.07" rpy="0 0.2617994 0" />
+      </joint>
+      <link name="camera_depth_frame" />
+      <joint name="camera_depth_joint" type="fixed">
+        <parent link="camera_link" />
+        <child link="camera_depth_frame" />
+        <origin xyz="0 0 0" rpy="0 0 0" />
+      </joint>
+      <link name="camera_depth_optical_frame" />
+      <joint name="camera_depth_optical_joint" type="fixed">
+        <parent link="camera_depth_frame" />
+        <child link="camera_depth_optical_frame" />
+        <origin xyz="0 0 0" rpy="${-pi/2} 0 ${-pi/2}" />
+      </joint>
+      <link name="camera_color_frame" />
+      <joint name="camera_color_joint" type="fixed">
+        <parent link="camera_link" />
+        <child link="camera_color_frame" />
+        <origin xyz="0 0 0" rpy="0 0 0" />
+      </joint>
+      <link name="camera_color_optical_frame" />
+      <joint name="camera_color_optical_joint" type="fixed">
+        <parent link="camera_color_frame" />
+        <child link="camera_color_optical_frame" />
+        <origin xyz="0 0 0" rpy="${-pi/2} 0 ${-pi/2}" />
+      </joint>
+    </xacro:if>
     <xacro:leg prefix="rear_left" xyz="-0.131 0.06 0.06" rpy="0 0 ${pi}" first_joint_offset="${pi}"
       third_joint_gear_correction_dir="-1.0" />

File: ros/src/wojtek_viz/urdf/wojtek_sim.urdf.xacro (robot description, xacro)
@@ -8,4 +8,7 @@
 <robot name="quadruped" xmlns:xacro="http://www.ros.org/wiki/xacro">
   <xacro:include filename="$(find wojtek_description)/urdf/body.urdf.xacro" />
-  <xacro:wojtek_body />
+  <!-- In sim the robot model owns the camera extrinsics (ground truth) -
+       robot_state_publisher latches base_link->camera_link->optical frames
+       matching the MJCF render camera; see wojtek_viz/camera_spec.py. -->
+  <xacro:wojtek_body with_camera="true" />
 </robot>
