Commit message: fix(ros): the IMU sits upright, so stop rotating its data by 180 deg
body.urdf.xacro declared imu_joint at rpy 0 pi 0, left over from the
previous IMU. The Adafruit 5543 that replaced it sits upright: measured
at rest on the robot, linear_acceleration.z = +10.05 m/s2, and
imu_i2c.cpp reads the chip axes straight into x/y/z with no remap. So
what arrives on /imu_sensor_broadcaster/imu is already base_link.

policy_node compensated a mount that is not there, which negated gravity
and the gyro's x and z. Nothing noticed for months because every policy
deployed so far had a 40-dim observation without the IMU. The first one
that reads it, terrain_blind v41 (46-dim, gyro + gravity), was handed a
gravity vector pointing up -- it believed the robot hung upside down and
fought that at 50 Hz. Measured on the bench, disarmed, with the robot
perfectly still:

  target std 0.489 rad, p-p 0.98 rad, dominant 25.0 Hz (half the policy
  rate: the output flipped every single step)

Feeding the same frozen observation to the previous policy produced a
dead-flat target, and negating gravity alone settled v41 completely, so
the sensors and the data path were never the problem. After this change,
on the same bench: target std 0.0002 rad, p-p 0.0008 rad, and the step
the servos take at arming is 0.10 rad (4.1 Nm against a 32 Nm cap).

The value lives in three places -- the model, the launch, and the
simulation's plugin -- and they drifted apart when the sensor was
swapped. All three are set to identity here. The simulation's copy
matters as much as the robot's: it deliberately emulated the flipped
mount so policy_node's compensation was exercised, which is exactly why
the simulation walked while the robot shook.

Co-Authored-By: Claude Opus 5 <noreply@anthropic.com>
Claude-Session: REDACTED

File: ros/src/wojtek_description/urdf/body.urdf.xacro (robot description, xacro)
@@ -41,8 +41,15 @@
     </joint>
     <link name="imu_link" />
+    <!-- The Adafruit 5543 sits UPRIGHT: measured at rest on the robot,
+         linear_acceleration.z = +10.05 m/s2, and imu_i2c.cpp reads the chip
+         axes straight into x/y/z with no remap. The rpy 0 pi 0 that stood
+         here was left over from the previous IMU and made policy_node flip
+         gravity and the gyro's x/z, which stayed invisible until a policy
+         actually read the IMU (terrain_blind v41). That one then fought a
+         robot it believed was upside down. -->
     <joint name="imu_joint" type="fixed">
       <parent link="base_link" />
       <child link="imu_link" />
-      <origin xyz="0.0 0.0 0.1" rpy=" 0.0 ${pi} 0.0" />
+      <origin xyz="0.0 0.0 0.1" rpy="0.0 0.0 0.0" />
     </joint>
     <xacro:if value="${with_camera}">

File: ros/src/wojtek_pc/urdf/wojtek_sim.urdf.xacro (robot description, xacro)
@@ -86,7 +86,10 @@
         <param name="initial_pose">$(arg boot_pose)</param>
         <param name="dry_run">$(arg dry_run)</param>
-        <!-- Emulate the physical mount (URDF imu_joint: rpy 0 pi 0) so
-             policy_node's imu_mount_rpy is exercised rather than bypassed. -->
-        <param name="imu_mount_rpy">0 3.141592653589793 0</param>
+        <!-- Emulate the physical mount (URDF imu_joint: rpy 0 0 0, i.e. the
+             sensor is upright, see body.urdf.xacro). The simulated IMU must
+             keep matching the real one: while this said pi and the hardware
+             said 0, the simulation exercised a compensation the robot did
+             not need, and walked while the robot shook. -->
+        <param name="imu_mount_rpy">0 0 0</param>
       </xacro:unless>
     </hardware>
