Commit message: fix(v627): the legs' URDF turns its hips and knees the way the drives do; the map carries the model's signs
On the robot's first stand-up (2026-10-23) four drives turned the wrong way:
the hip of rear_left and front_right, the knee of rear_right and front_left.
The v6.27 URDF took its joint axes from the training model (hips about the
mount's dir, knees about -dir, the mechanism mirrored between front and
rear) and the wojtek_v2 profile used the identity map, so those four joints
reached the drives with the opposite sign. The drives did not change with
the legs: the MD80 interface writes URDF joint angles, and the stock URDF
fixes their sense of rotation (+z of every hip and knee joint frame).

- leg_v627.urdf.xacro: hip and knee axes +z like the stock leg, limits in
  that sense.
- joint_map_v627.yaml replaces joint_map_identity.yaml: sign dir on the
  hips, -dir on the knees, offsets zero (both models share the zero pose).
- real_io: the v6.27 passive table is fitted in the model's convention, so
  the lever goes through the map and the result comes back through it
  (RobotPoses.passive_convention; the stock table stays URDF-to-URDF).
- tests: wojtek_bringup's test_leg_axes_follow_the_drives (every variant's
  actuated axes equal the stock URDF's in base_link; pins the stock axes),
  test_robots checks the four flipped signs and zero offsets.

Co-Authored-By: Claude Fable 5.1 <noreply@anthropic.com>

File: ros/src/wojtek_description/urdf/leg_v627.urdf.xacro (robot description, xacro)
@@ -10,7 +10,9 @@
        not change. From the second joint on it differs from the stock leg in
        three ways that matter to whoever drives it:
-         - Joint angles are the MuJoCo model's angles. The stock leg has
-           gear-correction offsets in its URDF and joint_map.yaml to undo
-           them; this leg needs the identity map.
+         - No gear-correction offsets: the zero pose is the training
+           model's. The sense of rotation of the hip and knee joints is the
+           drives' (+z of the joint frame, like the stock leg), which on two
+           joints per leg is the opposite of the model's; joint_map_v627.yaml
+           carries those signs.
          - Front and rear legs are mounted mirrored (knees point at each
            other), so the rear legs' second and third joints run negative.
@@ -58,8 +60,17 @@
       <child link="${prefix}_third_link" />
       <origin xyz="0.064 0 0.0668000048" rpy="0 0 ${pi if rear else 0.0}" />
-      <axis xyz="0 0 ${dir}" />
+      <!-- Axis +z of the joint frame on every leg, like the stock legs: the
+           drives did not change with the legs, and the MD80 interface writes
+           URDF joint angles to them, so the URDF keeps the drives' sense of
+           rotation. The mechanism's own convention (the training model,
+           wojtek.xml: hips about +-y by the dir of the mount) differs on
+           this joint by `dir`; joint_map_v627.yaml carries that sign, with
+           the limits below written in the URDF's (the drives') sense.
+           Seen on the robot 2026-10-23: with the model's axes here and the
+           identity map, four drives turned the wrong way at stand-up. -->
+      <axis xyz="0 0 1" />
       <limit effort="22" velocity="20"
-        lower="${min(lim*1.53588974, lim*2.69478837)}"
-        upper="${max(lim*1.53588974, lim*2.69478837)}" />
+        lower="${min(dir*lim*1.53588974, dir*lim*2.69478837)}"
+        upper="${max(dir*lim*1.53588974, dir*lim*2.69478837)}" />
     </joint>
     <!-- Crank (dzwignia), L2 = 33.0 mm, on the hip axis. -->
@@ -72,8 +83,10 @@
       <child link="${prefix}_fourth_link" />
       <origin xyz="0 0 0" rpy="0 0 0" />
-      <axis xyz="0 0 ${-dir}" />
+      <!-- Drives' sense again (see the second joint); the model's axis is
+           -dir here, so the map's sign for this joint is -dir. -->
+      <axis xyz="0 0 1" />
       <limit effort="22" velocity="20"
-        lower="${min(lim*0.244346095, lim*2.83266938)}"
-        upper="${max(lim*0.244346095, lim*2.83266938)}" />
+        lower="${min(-dir*lim*0.244346095, -dir*lim*2.83266938)}"
+        upper="${max(-dir*lim*0.244346095, -dir*lim*2.83266938)}" />
     </joint>
     <!-- Rod (wodzik), L4 = 291.0 mm, passive. -->

Commit message: fix(v627): the knee drives turn the same way on every leg, not mirrored like the stock ones
Second stand-up on the robot (2026-10-23): hips right, the levers of the
right legs backwards. The previous commit gave the v6.27 knees the stock
URDF's mirrored sense (left legs about +y of the body, right legs about -y),
which is the body's hip drives' arrangement, not the knee drives' on the
new thighs: those sit the same way on every leg and all four turn about +y.
The URDF knee axis is now lim*dir in the leg frame (+y of the body on all
four legs), every knee folds at -0.244 and stands near -2.0 in the URDF,
and the map's knee sign is -lim: +1 on the rear legs, -1 on the front
ones (against the model's -dir axes).

The bringup axes test now checks the body's drives (abduction, hip)
against the stock URDF and pins the measured knee sense per variant.

Co-Authored-By: Claude Fable 5.1 <noreply@anthropic.com>

File: ros/src/wojtek_description/urdf/leg_v627.urdf.xacro (robot description, xacro)
@@ -83,10 +83,14 @@
       <child link="${prefix}_fourth_link" />
       <origin xyz="0 0 0" rpy="0 0 0" />
-      <!-- Drives' sense again (see the second joint); the model's axis is
-           -dir here, so the map's sign for this joint is -dir. -->
-      <axis xyz="0 0 1" />
-      <limit effort="22" velocity="20"
-        lower="${min(-dir*lim*0.244346095, -dir*lim*2.83266938)}"
-        upper="${max(-dir*lim*0.244346095, -dir*lim*2.83266938)}" />
+      <!-- Drives' sense again, but NOT the stock leg's: the stock knee
+           drives are mirrored left/right (left about +y, right about -y of
+           the body), the v6.37a knee drives sit the same way on every leg
+           and all four turn about +y of the body (measured on the robot
+           2026-10-23: with the stock mirroring the right levers ran
+           backwards). In the leg frame that is lim*dir; against the model's
+           -dir the map's sign is -lim: +1 rear, -1 front. Every knee then
+           folds at -0.244 and stands at about -2.0 in the URDF. -->
+      <axis xyz="0 0 ${lim*dir}" />
+      <limit effort="22" velocity="20" lower="-2.83266938" upper="-0.244346095" />
     </joint>
     <!-- Rod (wodzik), L4 = 291.0 mm, passive. -->

Commit message: Revert "fix(v627): the knee drives turn the same way on every leg, not mirrored like the stock ones"
This reverts commit 0e4c5fff. Measured by hand on the robot (2026-10-23,
drives disabled, encoders streaming, each leg straightened as if
standing): levers rear_left -1.67, rear_right +2.11, front_right +1.37,
front_left -2.09 rad; hips rear_left -0.23, rear_right +0.53, front_right
+0.58, front_left -0.34 rad. Left legs negative, right legs positive on
both joints: the knee drives ARE mirrored left/right like the stock ones,
and the map of 4719f875 (hip sign dir, knee sign -dir) is the measured one.
The second stand-up that looked like the right levers running backwards
was a zero taken with one lever off its folding stop. The measurement is
recorded in the bringup axes test's docstring.

Co-Authored-By: Claude Fable 5.1 <noreply@anthropic.com>

File: ros/src/wojtek_description/urdf/leg_v627.urdf.xacro (robot description, xacro)
@@ -83,14 +83,10 @@
       <child link="${prefix}_fourth_link" />
       <origin xyz="0 0 0" rpy="0 0 0" />
-      <!-- Drives' sense again, but NOT the stock leg's: the stock knee
-           drives are mirrored left/right (left about +y, right about -y of
-           the body), the v6.37a knee drives sit the same way on every leg
-           and all four turn about +y of the body (measured on the robot
-           2026-10-23: with the stock mirroring the right levers ran
-           backwards). In the leg frame that is lim*dir; against the model's
-           -dir the map's sign is -lim: +1 rear, -1 front. Every knee then
-           folds at -0.244 and stands at about -2.0 in the URDF. -->
-      <axis xyz="0 0 ${lim*dir}" />
-      <limit effort="22" velocity="20" lower="-2.83266938" upper="-0.244346095" />
+      <!-- Drives' sense again (see the second joint); the model's axis is
+           -dir here, so the map's sign for this joint is -dir. -->
+      <axis xyz="0 0 1" />
+      <limit effort="22" velocity="20"
+        lower="${min(-dir*lim*0.244346095, -dir*lim*2.83266938)}"
+        upper="${max(-dir*lim*0.244346095, -dir*lim*2.83266938)}" />
     </joint>
     <!-- Rod (wodzik), L4 = 291.0 mm, passive. -->
