Commit message: feat(sim): tau_ff channel in the MuJoCo plant + base-collider and session fixes
Everything it took to run the tau_ff policy (wojtek-quiet-locomotion)
faithfully in the simulation, plus the bugs that surfaced on the way:

  * tau_ff channel (the feature): the MuJoCo plant now accepts
    [position, effort] command interfaces like the MD80 driver, exports
    the effort command, clamps the head to +-tau_ff_scale and applies it
    via qfrc_applied on the actuated dofs -- exactly the training env's
    model (servo clamped at max_torque - scale, head clamped separately).
    wojtek_sim.urdf.xacro gets tau_ff/tau_ff_scale args wired from the
    policy contract; launch_common passes the scale to the sim xacro
    (the real drive keeps taking only the summed cap). Without this,
    forward_effort_controller failed to activate and a tau_ff policy ran
    with half its control authority missing.

  * base collider fix (build_model.py, regenerated wojtek_mjx.xml): the
    chessboard base boxes were centered at body z=0 while the measured
    base mesh spans z 0..0.12 -- the boxes stuck 5 cm below the belly,
    so a lying robot rested on a phantom box and hovered. Boxes now sit
    on top of z=0 (lying base height 0.011 m, was ~0.05). The explicit
    base inertial is deliberately untouched: existing policies trained
    against it. This phantom also affected training-time falls/lying.

  * stale model copy: wojtek_pc/config/wojtek_mjx.xml had been frozen at
    a pre-chessboard snapshot (base mass 10.0 vs 8.64, joint friction
    6x too high), so the plant simulated a different robot than the one
    policies train on. Refreshed from wojtek_description/mujoco; keeping
    the two in sync (or installing description's mujoco/ dir instead of
    copying) still wants a proper mechanism.

  * sim_viewer: pin geom groups 0-2 and disable island coloring -- the
    passive viewer came up showing collision primitives over the meshes
    and repainting bodies by contact island.

  * dev.sh/sim.sh: reuse a running container instead of `compose up`
    (which silently RECREATES it when the compose stack differs, killing
    the session inside and dropping the build overlay -- observed live),
    and select the GPU overlay only when nvidia-smi actually works, not
    merely when the runtime is registered.

Operational note, not in code: with a soft-kp policy the sim rehearsal
must boot folded (sim.sh boot_pose:=folded). Zeroing a standing plant
bakes ~0.24 rad of gravity sag into the offsets, the policy then sees
shifted observations and stands grotesquely splayed while RViz disagrees
with the physics. Folded zeroing corrects 0.022 rad. The 0.15 rad
max_arm_jump_rad gate also needs raising for kp=20 policies (0.35 used
here) -- the same will bite the real robot.

MJX-side validation (run.sh check --gpu / test-slow) still pending: the
local venv has no jax. Plain-MuJoCo check passes (stand z 0.129->0.124,
closure 0.84 mm); test_sim_xacro passes.

Co-Authored-By: Claude Fable 5 <noreply@anthropic.com>
Claude-Session: https://claude.ai/code/session_01UAmAj41RXCstzXSnEGJmjs

File: ros/src/wojtek_pc/urdf/wojtek_sim.urdf.xacro (robot description, xacro)
@@ -26,4 +26,10 @@
   <xacro:arg name="kd" default="1.6" />
   <xacro:arg name="max_torque" default="9.0" />
+  <!-- Feed-forward torque channel, wired from the policy contract like the
+       real xacro's tau_ff. max_torque is the DRIVE cap (pd max_torque +
+       tau_ff_scale, see launch_common); the plugin clamps the servo and the
+       head separately, as the training sim does. -->
+  <xacro:arg name="tau_ff" default="false" />
+  <xacro:arg name="tau_ff_scale" default="0.0" />
   <xacro:arg name="hw" default="mock" />
   <!-- Physics scene for hw:=mujoco. The launch resolves this from this
@@ -50,7 +56,10 @@
        gains travel as params so the mujoco plugin can write them into the
        actuators; the mock ignores them. -->
-  <xacro:macro name="wojtek_sim_joint" params="name kp kd max_torque">
+  <xacro:macro name="wojtek_sim_joint" params="name kp kd max_torque tau_ff:=false tau_ff_scale:=0.0">
     <joint name="${name}">
       <command_interface name="position" />
+      <xacro:if value="${tau_ff}">
+        <command_interface name="effort" />
+      </xacro:if>
       <state_interface name="position">
         <param name="initial_value">0.0</param>
@@ -65,4 +74,5 @@
       <param name="ddq_kd">${kd}</param>
       <param name="max_torque">${max_torque}</param>
+      <param name="tau_ff_scale">${tau_ff_scale}</param>
     </joint>
   </xacro:macro>
@@ -94,16 +104,16 @@
       </xacro:unless>
     </hardware>
-    <xacro:wojtek_sim_joint name="front_left_first_joint" kp="$(arg kp)" kd="$(arg kd)" max_torque="$(arg max_torque)" />
-    <xacro:wojtek_sim_joint name="front_left_second_joint" kp="$(arg kp)" kd="$(arg kd)" max_torque="$(arg max_torque)" />
-    <xacro:wojtek_sim_joint name="front_left_third_joint" kp="$(arg kp)" kd="$(arg kd)" max_torque="$(arg max_torque)" />
-    <xacro:wojtek_sim_joint name="front_right_first_joint" kp="$(arg kp)" kd="$(arg kd)" max_torque="$(arg max_torque)" />
-    <xacro:wojtek_sim_joint name="front_right_second_joint" kp="$(arg kp)" kd="$(arg kd)" max_torque="$(arg max_torque)" />
-    <xacro:wojtek_sim_joint name="front_right_third_joint" kp="$(arg kp)" kd="$(arg kd)" max_torque="$(arg max_torque)" />
-    <xacro:wojtek_sim_joint name="rear_right_first_joint" kp="$(arg kp)" kd="$(arg kd)" max_torque="$(arg max_torque)" />
-    <xacro:wojtek_sim_joint name="rear_right_second_joint" kp="$(arg kp)" kd="$(arg kd)" max_torque="$(arg max_torque)" />
-    <xacro:wojtek_sim_joint name="rear_right_third_joint" kp="$(arg kp)" kd="$(arg kd)" max_torque="$(arg max_torque)" />
-    <xacro:wojtek_sim_joint name="rear_left_first_joint" kp="$(arg kp)" kd="$(arg kd)" max_torque="$(arg max_torque)" />
-    <xacro:wojtek_sim_joint name="rear_left_second_joint" kp="$(arg kp)" kd="$(arg kd)" max_torque="$(arg max_torque)" />
-    <xacro:wojtek_sim_joint name="rear_left_third_joint" kp="$(arg kp)" kd="$(arg kd)" max_torque="$(arg max_torque)" />
+    <xacro:wojtek_sim_joint name="front_left_first_joint" kp="$(arg kp)" kd="$(arg kd)" max_torque="$(arg max_torque)" tau_ff="$(arg tau_ff)" tau_ff_scale="$(arg tau_ff_scale)" />
+    <xacro:wojtek_sim_joint name="front_left_second_joint" kp="$(arg kp)" kd="$(arg kd)" max_torque="$(arg max_torque)" tau_ff="$(arg tau_ff)" tau_ff_scale="$(arg tau_ff_scale)" />
+    <xacro:wojtek_sim_joint name="front_left_third_joint" kp="$(arg kp)" kd="$(arg kd)" max_torque="$(arg max_torque)" tau_ff="$(arg tau_ff)" tau_ff_scale="$(arg tau_ff_scale)" />
+    <xacro:wojtek_sim_joint name="front_right_first_joint" kp="$(arg kp)" kd="$(arg kd)" max_torque="$(arg max_torque)" tau_ff="$(arg tau_ff)" tau_ff_scale="$(arg tau_ff_scale)" />
+    <xacro:wojtek_sim_joint name="front_right_second_joint" kp="$(arg kp)" kd="$(arg kd)" max_torque="$(arg max_torque)" tau_ff="$(arg tau_ff)" tau_ff_scale="$(arg tau_ff_scale)" />
+    <xacro:wojtek_sim_joint name="front_right_third_joint" kp="$(arg kp)" kd="$(arg kd)" max_torque="$(arg max_torque)" tau_ff="$(arg tau_ff)" tau_ff_scale="$(arg tau_ff_scale)" />
+    <xacro:wojtek_sim_joint name="rear_right_first_joint" kp="$(arg kp)" kd="$(arg kd)" max_torque="$(arg max_torque)" tau_ff="$(arg tau_ff)" tau_ff_scale="$(arg tau_ff_scale)" />
+    <xacro:wojtek_sim_joint name="rear_right_second_joint" kp="$(arg kp)" kd="$(arg kd)" max_torque="$(arg max_torque)" tau_ff="$(arg tau_ff)" tau_ff_scale="$(arg tau_ff_scale)" />
+    <xacro:wojtek_sim_joint name="rear_right_third_joint" kp="$(arg kp)" kd="$(arg kd)" max_torque="$(arg max_torque)" tau_ff="$(arg tau_ff)" tau_ff_scale="$(arg tau_ff_scale)" />
+    <xacro:wojtek_sim_joint name="rear_left_first_joint" kp="$(arg kp)" kd="$(arg kd)" max_torque="$(arg max_torque)" tau_ff="$(arg tau_ff)" tau_ff_scale="$(arg tau_ff_scale)" />
+    <xacro:wojtek_sim_joint name="rear_left_second_joint" kp="$(arg kp)" kd="$(arg kd)" max_torque="$(arg max_torque)" tau_ff="$(arg tau_ff)" tau_ff_scale="$(arg tau_ff_scale)" />
+    <xacro:wojtek_sim_joint name="rear_left_third_joint" kp="$(arg kp)" kd="$(arg kd)" max_torque="$(arg max_torque)" tau_ff="$(arg tau_ff)" tau_ff_scale="$(arg tau_ff_scale)" />
     <!-- One component carries both the joints and the IMU, unlike the real
          robot where they are separate drivers on separate buses: the plugin

Commit message: fix(sim): export the tau_ff effort channel from the ros2_control sim plant
a5cefdd carried the tau_ff head to the real robot and put its sim parity
into mujoco_sim_node, which the sim bringup no longer uses. The live sim
is the ros2_control plant, and it kept exporting position-only commands.
The launch passes tau_ff:=true to both xacros and spawns
forward_effort_controller for both bringups, so with a tau_ff policy
(the pinned default since quiet-locomotion@553795b) the sim spawner died
failing to claim the twelve effort interfaces and the session silently
ran PD-only, under hw:=mock and hw:=mujoco alike.

- wojtek_sim.urdf.xacro takes tau_ff and conditionally adds the effort
  command interface per joint, mirroring the real macro.
- MujocoHardwareInterface accepts a [position, effort] pair, exports the
  effort command, and writes it to the plant every cycle; non-finite
  falls back to 0 (pure PD), the same guard the MD80 driver runs.
- MujocoPlant::setFeedForward applies the torque through qfrc_applied,
  the mechanism the training env uses, zeroed in dry run.
- test_sim_xacro.py gains the tau_ff:=true comparison this drift
  slipped past; test_mujoco_plant.cpp pins the torque path and its
  dry-run guard.

Validated: test_sim_xacro.py passes (6) under a local xacro venv with a
stubbed ament index, and the new test fails on the pre-fix xacro. The
plant test's 0.1 rad threshold was measured at 0.23 rad of margin with
a Python replica of the plant on the stand-in model. The C++ compiles
only in the ROS gate (no ROS on this machine); run it before robot use.

Co-Authored-By: Claude Fable 5 <noreply@anthropic.com>

File: ros/src/wojtek_pc/urdf/wojtek_sim.urdf.xacro (robot description, xacro)
@@ -26,4 +26,7 @@
   <xacro:arg name="kd" default="1.6" />
   <xacro:arg name="max_torque" default="9.0" />
+  <!-- Mirrors the real xacro's effort channel, the feed-forward torque a
+       tau_ff policy adds on top of the servo. -->
+  <xacro:arg name="tau_ff" default="false" />
   <xacro:arg name="hw" default="mock" />
   <!-- Physics scene for hw:=mujoco. The launch resolves this from this
@@ -47,10 +50,14 @@
   <xacro:wojtek_body with_camera="true" />
   <!-- Same interface set as wojtek_bringup's wojtek_joint macro: a position
-       command (impedance target) and position/velocity/effort states. The
-       gains travel as params so the mujoco plugin can write them into the
-       actuators; the mock ignores them. -->
-  <xacro:macro name="wojtek_sim_joint" params="name kp kd max_torque">
+       command (impedance target) and position/velocity/effort states, plus
+       the effort command tau_ff adds. The gains travel as params so the
+       mujoco plugin can write them into the actuators; the mock ignores
+       them. -->
+  <xacro:macro name="wojtek_sim_joint" params="name kp kd max_torque tau_ff:=false">
     <joint name="${name}">
       <command_interface name="position" />
+      <xacro:if value="${tau_ff}">
+        <command_interface name="effort" />
+      </xacro:if>
       <state_interface name="position">
         <param name="initial_value">0.0</param>
@@ -94,16 +101,16 @@
       </xacro:unless>
     </hardware>
-    <xacro:wojtek_sim_joint name="front_left_first_joint" kp="$(arg kp)" kd="$(arg kd)" max_torque="$(arg max_torque)" />
-    <xacro:wojtek_sim_joint name="front_left_second_joint" kp="$(arg kp)" kd="$(arg kd)" max_torque="$(arg max_torque)" />
-    <xacro:wojtek_sim_joint name="front_left_third_joint" kp="$(arg kp)" kd="$(arg kd)" max_torque="$(arg max_torque)" />
-    <xacro:wojtek_sim_joint name="front_right_first_joint" kp="$(arg kp)" kd="$(arg kd)" max_torque="$(arg max_torque)" />
-    <xacro:wojtek_sim_joint name="front_right_second_joint" kp="$(arg kp)" kd="$(arg kd)" max_torque="$(arg max_torque)" />
-    <xacro:wojtek_sim_joint name="front_right_third_joint" kp="$(arg kp)" kd="$(arg kd)" max_torque="$(arg max_torque)" />
-    <xacro:wojtek_sim_joint name="rear_right_first_joint" kp="$(arg kp)" kd="$(arg kd)" max_torque="$(arg max_torque)" />
-    <xacro:wojtek_sim_joint name="rear_right_second_joint" kp="$(arg kp)" kd="$(arg kd)" max_torque="$(arg max_torque)" />
-    <xacro:wojtek_sim_joint name="rear_right_third_joint" kp="$(arg kp)" kd="$(arg kd)" max_torque="$(arg max_torque)" />
-    <xacro:wojtek_sim_joint name="rear_left_first_joint" kp="$(arg kp)" kd="$(arg kd)" max_torque="$(arg max_torque)" />
-    <xacro:wojtek_sim_joint name="rear_left_second_joint" kp="$(arg kp)" kd="$(arg kd)" max_torque="$(arg max_torque)" />
-    <xacro:wojtek_sim_joint name="rear_left_third_joint" kp="$(arg kp)" kd="$(arg kd)" max_torque="$(arg max_torque)" />
+    <xacro:wojtek_sim_joint name="front_left_first_joint" kp="$(arg kp)" kd="$(arg kd)" max_torque="$(arg max_torque)" tau_ff="$(arg tau_ff)" />
+    <xacro:wojtek_sim_joint name="front_left_second_joint" kp="$(arg kp)" kd="$(arg kd)" max_torque="$(arg max_torque)" tau_ff="$(arg tau_ff)" />
+    <xacro:wojtek_sim_joint name="front_left_third_joint" kp="$(arg kp)" kd="$(arg kd)" max_torque="$(arg max_torque)" tau_ff="$(arg tau_ff)" />
+    <xacro:wojtek_sim_joint name="front_right_first_joint" kp="$(arg kp)" kd="$(arg kd)" max_torque="$(arg max_torque)" tau_ff="$(arg tau_ff)" />
+    <xacro:wojtek_sim_joint name="front_right_second_joint" kp="$(arg kp)" kd="$(arg kd)" max_torque="$(arg max_torque)" tau_ff="$(arg tau_ff)" />
+    <xacro:wojtek_sim_joint name="front_right_third_joint" kp="$(arg kp)" kd="$(arg kd)" max_torque="$(arg max_torque)" tau_ff="$(arg tau_ff)" />
+    <xacro:wojtek_sim_joint name="rear_right_first_joint" kp="$(arg kp)" kd="$(arg kd)" max_torque="$(arg max_torque)" tau_ff="$(arg tau_ff)" />
+    <xacro:wojtek_sim_joint name="rear_right_second_joint" kp="$(arg kp)" kd="$(arg kd)" max_torque="$(arg max_torque)" tau_ff="$(arg tau_ff)" />
+    <xacro:wojtek_sim_joint name="rear_right_third_joint" kp="$(arg kp)" kd="$(arg kd)" max_torque="$(arg max_torque)" tau_ff="$(arg tau_ff)" />
+    <xacro:wojtek_sim_joint name="rear_left_first_joint" kp="$(arg kp)" kd="$(arg kd)" max_torque="$(arg max_torque)" tau_ff="$(arg tau_ff)" />
+    <xacro:wojtek_sim_joint name="rear_left_second_joint" kp="$(arg kp)" kd="$(arg kd)" max_torque="$(arg max_torque)" tau_ff="$(arg tau_ff)" />
+    <xacro:wojtek_sim_joint name="rear_left_third_joint" kp="$(arg kp)" kd="$(arg kd)" max_torque="$(arg max_torque)" tau_ff="$(arg tau_ff)" />
     <!-- One component carries both the joints and the IMU, unlike the real
          robot where they are separate drivers on separate buses: the plugin
